File: qsbc.kicad_pcb (KiCad board)
At the start: 8 copper layers, 80 x 80 mm, 371 parts, among them J1001 1-2199230-6, J501 USB_C_Receptacle_USB2.0, J502 USB_C_Receptacle_USB2.0, J503 USB_C_Receptacle_USB2.0, J504 USB_C_Receptacle_USB2.0, J601 ARJM11D7-502-AB-EW2, J701 Micro_SD_Card_Det1, J801 Conn_ARM_JTAG_SWD_10, SW401 SW_Push, SW801 SW_DIP_x02, U1001 SI52112-B5-GM2, U1002 74LVC1G07, U1003 74LVC1G07, U201 MIMX8MM6DVTLZAA, U202 MT40A1G16KD-062E, U401 BD71847MWV, U501 74LVC1G04, U502 74LVC1G04, U503 NX5P3363, U504 TUSB320LAI, U505 NX5P3363, U506 TUSB320LAI, U507 D5V0H1B2LP, U508 D5V0H1B2LP, U509 TPD4EUSB30, U510 TPD4EUSB30, U511 74LVC1G07, U512 74LVC1G07, U513 D5V0H1B2LP, U514 CH343P, U515 TPD4EUSB30, U516 INA231, U517 D5V0H1B2LP, U518 TS3USB221E, U519 TPD4EUSB30, U601 RTL8211FD, U602 TPD4EUSB30, U603 TPD4EUSB30, U701 TPD4EUSB30, U702 D5V0H1B2LP, U703 W25Q32JWZP, U704 SiP32431DR3, U705 TPD4EUSB30, Y1001 25MHz, Y401 Crystal, Y601 25MHz, Y801 24Mhz

Commit message: add inital ddr tool version, lots of routing work
Parts:
- removed FB501, FB502, FB503, FB504: FerriteBead, Resistor_SMD:R_0603_1608Metric
- removed TP201: TestPoint, TestPoint:TestPoint_Pad_D1.0mm
- added C149: 0.1uF, Capacitor_SMD:C_0402_1005Metric, F.Cu at (175.3, 62.7)
- added C150: 0.1uF, Capacitor_SMD:C_0402_1005Metric, F.Cu at (178.2, 62.7)
- added C84: 1uF, Capacitor_SMD:C_0402_1005Metric, F.Cu at (113.9, 93.7)
- added C85: 1uF, Capacitor_SMD:C_0402_1005Metric, F.Cu at (117.2, 101.7)
- added D3: LED_Green, LED_SMD:LED_0603_1608Metric, F.Cu at (165.3, 65.5)
- added D4: LED_Red, LED_SMD:LED_0603_1608Metric, F.Cu at (169.4, 65.5)
- added R103: 2.2K, Resistor_SMD:R_0402_1005Metric, F.Cu at (172.9, 65.2)
- added R48: 0R, Resistor_SMD:R_0402_1005Metric, F.Cu at (182.0, 37.5)
- added R49: 10K, Resistor_SMD:R_0402_1005Metric, F.Cu at (179.1, 37.5)
- added R98: 2.2K, Resistor_SMD:R_0402_1005Metric, F.Cu at (175.1, 60.7)
- added TP18: TestPoint, TestPoint:TestPoint_Pad_D1.0mm, F.Cu at (117.3, 91.7)
- added U32: 74LVC1G07, Package_TO_SOT_SMD:SOT-23-5, F.Cu at (171.0, 61.9)
- added U33: 74LVC1G07, Package_TO_SOT_SMD:SOT-23-5, F.Cu at (165.9, 61.9)
- added U4: NCP718BSN250T1G, Package_TO_SOT_SMD:SOT-23-5, F.Cu at (117.4, 94.7)
- C1: renamed from C201; footprint Capacitor_SMD:C_0201_0603Metric -> qsbc:C_0201_0603Metric; moved to B.Cu
- C119: renamed from C511; footprint Capacitor_SMD:C_0201_0603Metric -> qsbc:C_0201_0603Metric
- C12: renamed from C212; footprint Capacitor_SMD:C_0201_0603Metric -> qsbc:C_0201_0603Metric; moved to B.Cu
- C120: renamed from C512; footprint Capacitor_SMD:C_0201_0603Metric -> qsbc:C_0201_0603Metric
- C13: renamed from C301; footprint Capacitor_SMD:C_0201_0603Metric -> qsbc:C_0201_0603Metric
- C135: renamed from C609; value 27pF -> 14pF
- C137: renamed from C611; value 27pF -> 14pF
- C147: renamed from C801; value 12pF -> 14pF
- C148: renamed from C802; value 12pF -> 14pF
- C153: renamed from C1003; value 20pF -> 14pF
- C154: renamed from C1004; value 20pF -> 14pF
- C18: renamed from C306; footprint Capacitor_SMD:C_0201_0603Metric -> qsbc:C_0201_0603Metric
- C19: renamed from C307; footprint Capacitor_SMD:C_0201_0603Metric -> qsbc:C_0201_0603Metric
- C2: renamed from C202; moved to B.Cu
- C20: renamed from C308; footprint Capacitor_SMD:C_0201_0603Metric -> qsbc:C_0201_0603Metric
- C21: renamed from C309; footprint Capacitor_SMD:C_0201_0603Metric -> qsbc:C_0201_0603Metric
- C24: renamed from C312; footprint Capacitor_SMD:C_0201_0603Metric -> qsbc:C_0201_0603Metric
- C25: renamed from C313; footprint Capacitor_SMD:C_0201_0603Metric -> qsbc:C_0201_0603Metric
- C26: renamed from C314; footprint Capacitor_SMD:C_0201_0603Metric -> qsbc:C_0201_0603Metric
- C27: renamed from C315; footprint Capacitor_SMD:C_0201_0603Metric -> qsbc:C_0201_0603Metric
- C28: renamed from C316; footprint Capacitor_SMD:C_0201_0603Metric -> qsbc:C_0201_0603Metric
- C29: renamed from C317; footprint Capacitor_SMD:C_0201_0603Metric -> qsbc:C_0201_0603Metric
- C3: renamed from C203; moved to B.Cu
- C30: renamed from C318; footprint Capacitor_SMD:C_0201_0603Metric -> qsbc:C_0201_0603Metric
- C31: renamed from C319; footprint Capacitor_SMD:C_0201_0603Metric -> qsbc:C_0201_0603Metric
- C32: renamed from C320; footprint Capacitor_SMD:C_0201_0603Metric -> qsbc:C_0201_0603Metric
- C33: renamed from C321; footprint Capacitor_SMD:C_0201_0603Metric -> qsbc:C_0201_0603Metric
- C34: renamed from C322; footprint Capacitor_SMD:C_0201_0603Metric -> qsbc:C_0201_0603Metric
- C35: renamed from C323; footprint Capacitor_SMD:C_0201_0603Metric -> qsbc:C_0201_0603Metric
- C36: renamed from C324; footprint Capacitor_SMD:C_0201_0603Metric -> qsbc:C_0201_0603Metric
- C37: renamed from C325; footprint Capacitor_SMD:C_0201_0603Metric -> qsbc:C_0201_0603Metric
- C38: renamed from C326; footprint Capacitor_SMD:C_0201_0603Metric -> qsbc:C_0201_0603Metric
- C39: renamed from C327; footprint Capacitor_SMD:C_0201_0603Metric -> qsbc:C_0201_0603Metric
- C4: renamed from C204; moved to B.Cu
- C40: renamed from C328; footprint Capacitor_SMD:C_0201_0603Metric -> qsbc:C_0201_0603Metric
- C41: renamed from C329; footprint Capacitor_SMD:C_0201_0603Metric -> qsbc:C_0201_0603Metric
- C42: renamed from C330; footprint Capacitor_SMD:C_0201_0603Metric -> qsbc:C_0201_0603Metric
- C43: renamed from C331; footprint Capacitor_SMD:C_0201_0603Metric -> qsbc:C_0201_0603Metric
- C44: renamed from C332; footprint Capacitor_SMD:C_0201_0603Metric -> qsbc:C_0201_0603Metric
- C45: renamed from C333; footprint Capacitor_SMD:C_0201_0603Metric -> qsbc:C_0201_0603Metric
- C48: renamed from C336; footprint Capacitor_SMD:C_0201_0603Metric -> qsbc:C_0201_0603Metric
- C49: renamed from C337; footprint Capacitor_SMD:C_0201_0603Metric -> qsbc:C_0201_0603Metric
- C52: renamed from C340; footprint Capacitor_SMD:C_0201_0603Metric -> qsbc:C_0201_0603Metric
- C54: renamed from C342; footprint Capacitor_SMD:C_0201_0603Metric -> qsbc:C_0201_0603Metric
- C55: renamed from C343; footprint Capacitor_SMD:C_0201_0603Metric -> qsbc:C_0201_0603Metric
- C56: renamed from C344; footprint Capacitor_SMD:C_0201_0603Metric -> qsbc:C_0201_0603Metric
- C57: renamed from C345; footprint Capacitor_SMD:C_0201_0603Metric -> qsbc:C_0201_0603Metric
- C58: renamed from C346; footprint Capacitor_SMD:C_0201_0603Metric -> qsbc:C_0201_0603Metric
- C59: renamed from C347; footprint Capacitor_SMD:C_0201_0603Metric -> qsbc:C_0201_0603Metric
- C60: renamed from C348; footprint Capacitor_SMD:C_0201_0603Metric -> qsbc:C_0201_0603Metric
- C61: renamed from C349; footprint Capacitor_SMD:C_0201_0603Metric -> qsbc:C_0201_0603Metric
- C62: renamed from C350; footprint Capacitor_SMD:C_0201_0603Metric -> qsbc:C_0201_0603Metric
- C63: renamed from C351; footprint Capacitor_SMD:C_0201_0603Metric -> qsbc:C_0201_0603Metric
- C64: renamed from C352; footprint Capacitor_SMD:C_0201_0603Metric -> qsbc:C_0201_0603Metric
- C65: renamed from C353; footprint Capacitor_SMD:C_0201_0603Metric -> qsbc:C_0201_0603Metric
- C66: renamed from C354; footprint Capacitor_SMD:C_0201_0603Metric -> qsbc:C_0201_0603Metric
- C67: renamed from C355; footprint Capacitor_SMD:C_0201_0603Metric -> qsbc:C_0201_0603Metric
- C68: renamed from C356; footprint Capacitor_SMD:C_0201_0603Metric -> qsbc:C_0201_0603Metric
- C69: renamed from C357; footprint Capacitor_SMD:C_0201_0603Metric -> qsbc:C_0201_0603Metric
- C8: renamed from C208; moved to B.Cu
- R1: renamed from R201; footprint Resistor_SMD:R_0201_0603Metric -> qsbc:R_0201_0603Metric; moved to B.Cu
- R10: renamed from R210; footprint Resistor_SMD:R_0201_0603Metric -> qsbc:R_0201_0603Metric; moved to B.Cu
- R2: renamed from R202; footprint Resistor_SMD:R_0201_0603Metric -> qsbc:R_0201_0603Metric; moved to B.Cu
- R29: renamed from R511; footprint Resistor_SMD:R_0201_0603Metric -> qsbc:R_0201_0603Metric
- R3: renamed from R203; footprint Resistor_SMD:R_0201_0603Metric -> qsbc:R_0201_0603Metric; moved to B.Cu
- R30: renamed from R512; footprint Resistor_SMD:R_0201_0603Metric -> qsbc:R_0201_0603Metric
- R33: renamed from R515; footprint Resistor_SMD:R_0201_0603Metric -> qsbc:R_0201_0603Metric
- R34: renamed from R516; footprint Resistor_SMD:R_0201_0603Metric -> qsbc:R_0201_0603Metric
- R35: renamed from R517; footprint Resistor_SMD:R_0201_0603Metric -> qsbc:R_0201_0603Metric
- R36: renamed from R518; footprint Resistor_SMD:R_0201_0603Metric -> qsbc:R_0201_0603Metric
- R4: renamed from R204; footprint Resistor_SMD:R_0201_0603Metric -> qsbc:R_0201_0603Metric; moved to B.Cu
- R6: renamed from R206; footprint Resistor_SMD:R_0402_1005Metric -> qsbc:R_0201_0603Metric; moved to B.Cu
- R7: renamed from R207; footprint Resistor_SMD:R_0402_1005Metric -> qsbc:R_0201_0603Metric; moved to B.Cu
- R8: renamed from R208; footprint Resistor_SMD:R_0402_1005Metric -> qsbc:R_0201_0603Metric; moved to B.Cu
- R9: renamed from R209; footprint Resistor_SMD:R_0402_1005Metric -> qsbc:R_0201_0603Metric; moved to B.Cu
- TP2: renamed from TP202; footprint TestPoint:TestPoint_Pad_D1.0mm -> qsbc:TestPoint_Pad_D0.4mm; moved to B.Cu
- TP24: renamed from TP501; footprint TestPoint:TestPoint_Pad_D1.5mm -> TestPoint:TestPoint_Pad_D1.0mm
- moved C16 330.0 mm to (67.0, 52.2)
- moved C18 330.0 mm to (69.7, 50.1)
- moved C19 330.0 mm to (79.5, 49.7)
- moved C20 330.0 mm to (74.6, 49.9)
- moved C21 330.0 mm to (77.5, 47.9)
- moved C25 330.0 mm to (66.8, 54.1)
- moved C26 330.0 mm to (76.6, 55.2)
- moved C27 330.0 mm to (72.6, 48.2)
- moved C28 330.0 mm to (80.3, 46.2)
- moved C29 330.0 mm to (76.6, 53.4)
- moved C30 330.0 mm to (77.0, 51.7)
- moved C32 330.0 mm to (79.9, 47.9)
- moved C33 330.0 mm to (72.2, 50.1)
- moved C34 330.0 mm to (82.4, 47.9)
- moved C36 330.0 mm to (75.4, 46.2)
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- renumbered C210 to C10, C429 to C100, C430 to C101, C431 to C102, C432 to C103, C433 to C104, C434 to C105, C435 to C106, C436 to C107, C437 to C108, C501 to C109, C211 to C11, C502 to C110, C503 to C111, C504 to C112, C505 to C113, C506 to C114, C507 to C115, C508 to C116, C509 to C117, C510 to C118, C513 to C121, C514 to C122, C515 to C123, C516 to C124, C517 to C125, C518 to C126, C601 to C127, C602 to C128, C603 to C129, C604 to C130, C605 to C131, C606 to C132, C607 to C133, C608 to C134, C610 to C136, C612 to C138, C613 to C139, C302 to C14, C614 to C140, C701 to C141, C702 to C142, C703 to C143, C704 to C144, C705 to C145, C706 to C146, C303 to C15, C1001 to C151, C1002 to C152, C1005 to C155, C1006 to C156, C1007 to C157, C1008 to C158, C1009 to C159, C304 to C16, C1010 to C160, C1011 to C161, C1012 to C162, C1013 to C163, C1014 to C164, C305 to C17, C310 to C22, C311 to C23, C334 to C46, C335 to C47, C205 to C5, C338 to C50, C339 to C51, C341 to C53, C206 to C6, C207 to C7, C401 to C70, C402 to C71, C403 to C72, C404 to C73, C405 to C74, C406 to C75, C407 to C76, C408 to C77, C409 to C78, C410 to C79, C411 to C80, C412 to C81, C413 to C82, C414 to C83, C415 to C86, C416 to C87, C417 to C88, C418 to C89, C209 to C9, C419 to C90, C420 to C91, C421 to C92, C422 to C93, C423 to C94, C424 to C95, C425 to C96, C426 to C97, C427 to C98, C428 to C99, D501 to D1, D502 to D2, D1001 to D5, H101 to H1, H102 to H2, H103 to H3, H104 to H4, H1001 to H5, J501 to J1, J502 to J2, J503 to J3, J504 to J4, J601 to J5, J701 to J6, J801 to J7, J1001 to J8, L401 to L1, L402 to L2, L403 to L3, L404 to L4, L405 to L5, L406 to L6, R907 to R100, R908 to R101, R909 to R102, R910 to R104, R911 to R105, R912 to R106, R913 to R107, R914 to R108, R915 to R109, R211 to R11, R916 to R110, R917 to R111, R918 to R112, R919 to R113, R920 to R114, R1001 to R115, R1002 to R116, R1003 to R117, R1004 to R118, R1005 to R119, R212 to R12, R1006 to R120, R1007 to R121, R1008 to R122, R401 to R13, R402 to R14, R403 to R15, R404 to R16, R405 to R17, R406 to R18, R501 to R19, R502 to R20, R503 to R21, R504 to R22, R505 to R23, R506 to R24, R507 to R25, R508 to R26, R509 to R27, R510 to R28, R513 to R31, R514 to R32, R519 to R37, R520 to R38, R521 to R39, R522 to R40, R523 to R41, R524 to R42, R525 to R43, R526 to R44, R527 to R45, R528 to R46, R529 to R47, R205 to R5, R530 to R50, R531 to R51, R532 to R52, R601 to R53, R602 to R54, R603 to R55, R604 to R56, R605 to R57, R606 to R58, R607 to R59, R608 to R60, R609 to R61, R610 to R62, R611 to R63, R612 to R64, R613 to R65, R614 to R66, R615 to R67, R616 to R68, R617 to R69, R618 to R70, R619 to R71, R620 to R72, R621 to R73, R622 to R74, R623 to R75, R701 to R76, R702 to R77, R703 to R78, R704 to R79, R705 to R80, R801 to R81, R802 to R82, R803 to R83, R804 to R84, R805 to R85, R806 to R86, R807 to R87, R808 to R88, R809 to R89, R810 to R90, R811 to R91, R812 to R92, R901 to R93, R902 to R94, R903 to R95, R904 to R96, R905 to R97, R906 to R99, SW401 to SW1, SW801 to SW2, TP407 to TP10, TP408 to TP11, TP409 to TP12, TP410 to TP13, TP411 to TP14, TP412 to TP15, TP413 to TP16, TP414 to TP17, TP415 to TP19, TP416 to TP20, TP417 to TP21, TP418 to TP22, TP419 to TP23, TP801 to TP25, TP802 to TP26, TP803 to TP27, TP804 to TP28, TP805 to TP29, TP203 to TP3, TP401 to TP4, TP402 to TP5, TP403 to TP6, TP404 to TP7, TP405 to TP8, TP406 to TP9, U201 to U1, U506 to U10, U507 to U11, U508 to U12, U509 to U13, U510 to U14, U511 to U15, U512 to U16, U513 to U17, U514 to U18, U515 to U19, U202 to U2, U516 to U20, U517 to U21, U518 to U22, U519 to U23, U601 to U24, U602 to U25, U603 to U26, U701 to U27, U702 to U28, U703 to U29, U401 to U3, U704 to U30, U705 to U31, U1001 to U34, U1002 to U35, U1003 to U36, U501 to U5, U502 to U6, U503 to U7, U504 to U8, U505 to U9, Y401 to Y1, Y601 to Y2, Y801 to Y3, Y1001 to Y4
Connections:
- net /DDR/DRAM_ACT_N renamed /DDR/~{DRAM_ACT}
- net /DDR/DRAM_ALERT_N renamed /DDR/~{DRAM_ALERT}
- net /DDR/DRAM_CS0_N renamed /DDR/~{DRAM_CS0}
- net /DDR/DRAM_RESET_N renamed /DDR/~{DRAM_RESET}
- C10 pad 1: /DDR/NVCC_DRAM_1.2V -> /DDR/VDD_DRAM_1.2V
- C107 pad 1: /Misc/CLK_32K_OUT -> /Misc/NVCC_SNVS_1.8V
- C11 pad 1: /DDR/NVCC_DRAM_1.2V -> /DDR/VPP_2.5V
- C111 pad 1: VCC -> VDD_1.8V
- C112 pad 1: VCC -> VDD_1.8V
- C115 pad 1: VDD -> VDD_3.3V
- C116 pad 1: VDD -> VDD_3.3V
- C121 pad 1: VCC -> VDD_1.8V
- C122 pad 1: VCC -> VDD_1.8V
- C123 pad 1: VCC -> VDD_1.8V
- C124 pad 1: VDD -> VDD_3.3V
- C125 pad 1: VDD -> VDD_3.3V
- C126 pad 1: VDD -> VDD_3.3V
- C13 pad 1: /Misc/CLK_32K_OUT -> /Misc/NVCC_SNVS_1.8V
- C144 pad 1: VCC -> VDD_1.8V
- C145 pad 1: VDD -> VDD_3.3V
- C151 pad 1: VDD -> VDD_3.3V
- C152 pad 1: VDD -> VDD_3.3V
- C157 pad 1: VDD -> VDD_3.3V
- C158 pad 1: VDD -> VDD_3.3V
- C159 pad 1: VDD -> VDD_3.3V
- C160 pad 1: VDD -> VDD_3.3V
- C161 pad 1: VDD -> VDD_3.3V
- C162 pad 1: VDD -> VDD_3.3V
- C163 pad 1: VCC -> VDD_1.8V
- C164 pad 1: VCC -> VDD_1.8V
- C17 pad 1: /DDR/NVCC_DRAM_1.2V -> /DDR/VDD_DRAM_1.2V
- C2 pad 1: /DDR/NVCC_DRAM_1.2V -> /DDR/VDD_DRAM_1.2V
- C23 pad 1: /DDR/NVCC_DRAM_1.2V -> /DDR/VDD_DRAM_1.2V
- C27 pad 1: /DDR/NVCC_DRAM_1.2V -> /DDR/VDD_DRAM_1.2V
- C3 pad 1: /DDR/NVCC_DRAM_1.2V -> /DDR/VDD_DRAM_1.2V
- C32 pad 1: /DDR/NVCC_DRAM_1.2V -> /DDR/VDD_DRAM_1.2V
- C36 pad 1: /DDR/NVCC_DRAM_1.2V -> /DDR/VDD_DRAM_1.2V
- C4 pad 1: /DDR/NVCC_DRAM_1.2V -> /DDR/VDD_DRAM_1.2V
- C40 pad 1: /DDR/NVCC_DRAM_1.2V -> /DDR/VDD_DRAM_1.2V
- C42 pad 1: /DDR/NVCC_DRAM_1.2V -> /DDR/VDD_DRAM_1.2V
- C44 pad 1: /DDR/NVCC_DRAM_1.2V -> /DDR/VDD_DRAM_1.2V
- C45 pad 1: VCC -> VDD_1.8V
- C47 pad 1: VCC -> VDD_1.8V
- C48 pad 1: VCC -> VDD_1.8V
- C49 pad 1: VCC -> VDD_1.8V
- C5 pad 1: /DDR/NVCC_DRAM_1.2V -> /DDR/VDD_DRAM_1.2V
- C53 pad 1: VCC -> VDD_1.8V
- C54 pad 1: VCC -> VDD_1.8V
- C57 pad 1: VCC -> VDD_1.8V
- C58 pad 1: VDD -> VDD_3.3V
- C6 pad 1: /DDR/NVCC_DRAM_1.2V -> /DDR/VDD_DRAM_1.2V
- C60 pad 1: VCC -> VDD_1.8V
- C62 pad 1: VCC -> VDD_1.8V
- C63 pad 1: VCC -> VDD_1.8V
- C65 pad 1: VCC -> VDD_1.8V
- C68 pad 1: VCC -> VDD_1.8V
- C73 pad 1: VCC -> VDD_1.8V
- C74 pad 1: VDD -> VDD_3.3V
- C75 pad 1: VCC -> VDD_1.8V
- C8 pad 1: /DDR/NVCC_DRAM_1.2V -> /DDR/VDD_DRAM_1.2V
- C86 pad 1: /Misc/CLK_32K_OUT -> /Misc/NVCC_SNVS_1.8V
- C9 pad 1: /DDR/NVCC_DRAM_1.2V -> /DDR/VPP_2.5V
- C93 pad 1: /DDR/NVCC_DRAM_1.2V -> /DDR/VDD_DRAM_1.2V
- C94 pad 1: /DDR/NVCC_DRAM_1.2V -> /DDR/VDD_DRAM_1.2V
- C95 pad 1: VCC -> VDD_1.8V
- C96 pad 1: VCC -> VDD_1.8V
- C97 pad 1: VDD -> VDD_3.3V
- C98 pad 1: VDD -> VDD_3.3V
- J1 pad S1: Net-(FB501-Pad1) -> GND
- J2 pad S1: Net-(FB502-Pad1) -> GND
- J3 pad S1: Net-(FB503-Pad1) -> GND
- J4 pad S1: Net-(FB504-Pad1) -> GND
- J7 pad 1: VDD -> VDD_1.8V
- J8 pad 12: VDD -> VDD_3.3V
- J8 pad 14: VDD -> VDD_3.3V
- J8 pad 16: VDD -> VDD_3.3V
- J8 pad 18: VDD -> VDD_3.3V
- J8 pad 2: VDD -> VDD_3.3V
- J8 pad 4: VDD -> VDD_3.3V
- J8 pad 70: VDD -> VDD_3.3V
- J8 pad 72: VDD -> VDD_3.3V
- J8 pad 74: VDD -> VDD_3.3V
- L4 pad 2: VDD -> VDD_3.3V
- L5 pad 2: VCC -> VDD_1.8V
- L6 pad 2: /DDR/NVCC_DRAM_1.2V -> /DDR/VDD_DRAM_1.2V
- R100 pad 1: VCC -> VDD_1.8V
- R101 pad 1: VCC -> VDD_1.8V
- R102 pad 1: VCC -> VDD_1.8V
- R104 pad 1: VCC -> VDD_1.8V
- R105 pad 1: VCC -> VDD_1.8V
- R106 pad 1: VCC -> VDD_1.8V
- R107 pad 1: VCC -> VDD_1.8V
- R108 pad 1: VCC -> VDD_1.8V
- R109 pad 1: VCC -> VDD_1.8V
- R11 pad 2: /DDR/NVCC_DRAM_1.2V -> /DDR/VDD_DRAM_1.2V
- R110 pad 1: VCC -> VDD_1.8V
- R111 pad 1: VCC -> VDD_1.8V
- R112 pad 1: VCC -> VDD_1.8V
- R113 pad 1: VCC -> VDD_1.8V
- R114 pad 1: VCC -> VDD_1.8V
- R116 pad 1: VDD -> VDD_3.3V
- R117 pad 1: VDD -> VDD_3.3V
- R118 pad 1: VDD -> VDD_3.3V
- R119 pad 1: VDD -> VDD_3.3V
- R120 pad 1: VDD -> VDD_3.3V
- R121 pad 1: VCC -> VDD_1.8V
- R122 pad 1: VCC -> VDD_1.8V
- R17 pad 1: VCC -> VDD_1.8V
- R18 pad 1: /Misc/CLK_32K_OUT -> /Misc/NVCC_SNVS_1.8V
- R19 pad 1: VCC -> VDD_1.8V
- R20 pad 1: VCC -> VDD_1.8V
- R21 pad 1: VCC -> VDD_1.8V
- R22 pad 1: VCC -> VDD_1.8V
- R23 pad 1: VCC -> VDD_1.8V
- R24 pad 1: VCC -> VDD_1.8V
- R4 pad 2: /DDR/NVCC_DRAM_1.2V -> /DDR/VDD_DRAM_1.2V
- R41 pad 1: VCC -> VDD_1.8V
- R43 pad 1: VDD -> VDD_3.3V
- R46 pad 1: VDD -> VDD_3.3V
- R50 pad 1: /USB/USB3_VBUS -> Net-(R48-Pad2)
- R60 pad 1: VCC -> VDD_1.8V
- R61 pad 1: VCC -> VDD_1.8V
- R63 pad 1: VDD -> VDD_3.3V
- R64 pad 1: VDD -> VDD_3.3V
- R67 pad 1: VCC -> VDD_1.8V
- R79 pad 1: VCC -> VDD_1.8V
- R81 pad 1: /Misc/CLK_32K_OUT -> /Misc/NVCC_SNVS_1.8V
- R82 pad 1: /Misc/CLK_32K_OUT -> /Misc/NVCC_SNVS_1.8V
- R85 pad 1: /Misc/CLK_32K_OUT -> /Misc/NVCC_SNVS_1.8V
- R86 pad 1: VDD -> VDD_1.8V
- R88 pad 1: VDD -> VDD_1.8V
- R92 pad 1: VDD -> VDD_1.8V
- R93 pad 1: VCC -> VDD_1.8V
- R94 pad 1: VCC -> VDD_1.8V
- R95 pad 1: VCC -> VDD_1.8V
- R96 pad 1: VCC -> VDD_1.8V
- R97 pad 1: VCC -> VDD_1.8V
- R99 pad 1: VCC -> VDD_1.8V
- TP10 pad 1: /DDR/NVCC_DRAM_1.2V -> /DDR/VDD_DRAM_1.2V
- TP11 pad 1: /Misc/CLK_32K_OUT -> /Misc/NVCC_SNVS_1.8V
- TP8 pad 1: VDD -> VDD_3.3V
- TP9 pad 1: VCC -> VDD_1.8V
- U1 pad A14: unconnected-(U201-PadA14) -> GND
- U1 pad A15: unconnected-(U201-PadA15) -> GND
- U1 pad A16: unconnected-(U201-PadA16) -> GND
- U1 pad A17: unconnected-(U201-PadA17) -> GND
- U1 pad A18: unconnected-(U201-PadA18) -> GND
- U1 pad AB13: VCC -> VDD_1.8V
- U1 pad AF12: unconnected-(U201-PadAF12) -> /Peripherals/LED0
- U1 pad AG11: unconnected-(U201-PadAG11) -> /Peripherals/LED1
- U1 pad B14: unconnected-(U201-PadB14) -> GND
- U1 pad B15: unconnected-(U201-PadB15) -> GND
- U1 pad B16: unconnected-(U201-PadB16) -> GND
- U1 pad B17: unconnected-(U201-PadB17) -> GND
- U1 pad B18: unconnected-(U201-PadB18) -> GND
- U1 pad H10: VCC -> VDD_1.8V
- U1 pad J11: VCC -> VDD_1.8V
- U1 pad J12: VCC -> VDD_1.8V
- U1 pad J13: VCC -> VDD_1.8V
- U1 pad J22: /Misc/CLK_32K_OUT -> /Misc/NVCC_SNVS_1.8V
- U1 pad K19: VDD -> VDD_3.3V
- U1 pad K8: /DDR/NVCC_DRAM_1.2V -> /DDR/VDD_DRAM_1.2V
- U1 pad K9: /DDR/NVCC_DRAM_1.2V -> /DDR/VDD_DRAM_1.2V
- U1 pad L19: VCC -> VDD_1.8V
- U1 pad L9: /DDR/NVCC_DRAM_1.2V -> /DDR/VDD_DRAM_1.2V
- U1 pad M19: VCC -> VDD_1.8V
- U1 pad M9: /DDR/NVCC_DRAM_1.2V -> /DDR/VDD_DRAM_1.2V
- U1 pad N2: /DDR/DRAM_MTEST -> unconnected-(U1-PadN2)
- U1 pad N8: /DDR/NVCC_DRAM_1.2V -> /DDR/VDD_DRAM_1.2V
- U1 pad N9: /DDR/NVCC_DRAM_1.2V -> /DDR/VDD_DRAM_1.2V
- U1 pad P7: /DDR/NVCC_DRAM_1.2V -> /DDR/VDD_DRAM_1.2V
- U1 pad R8: /DDR/NVCC_DRAM_1.2V -> /DDR/VDD_DRAM_1.2V
- U1 pad R9: /DDR/NVCC_DRAM_1.2V -> /DDR/VDD_DRAM_1.2V
- U1 pad T19: VCC -> VDD_1.8V
- U1 pad T9: /DDR/NVCC_DRAM_1.2V -> /DDR/VDD_DRAM_1.2V
- U1 pad U19: VCC -> VDD_1.8V
- U1 pad U9: /DDR/NVCC_DRAM_1.2V -> /DDR/VDD_DRAM_1.2V
- U1 pad V19: VCC -> VDD_1.8V
- U1 pad V20: VCC -> VDD_1.8V
- U1 pad V8: /DDR/NVCC_DRAM_1.2V -> /DDR/VDD_DRAM_1.2V
- U1 pad V9: /DDR/NVCC_DRAM_1.2V -> /DDR/VDD_DRAM_1.2V
- U1 pad W12: VCC -> VDD_1.8V
- U1 pad W17: VCC -> VDD_1.8V
- U1 pad W18: VCC -> VDD_1.8V
- U1 pad Y10: VCC -> VDD_1.8V
- U10 pad 12: VDD -> VDD_3.3V
- U15 pad 5: VCC -> VDD_1.8V
- U16 pad 5: VCC -> VDD_1.8V
- U18 pad 3: VDD -> VDD_3.3V
- U18 pad 6: VDD -> VDD_3.3V
- U18 pad 9: VDD -> VDD_3.3V
- U2 pad A1: /DDR/NVCC_DRAM_1.2V -> /DDR/VDD_DRAM_1.2V
- U2 pad A3: /DDR/DRAM_D08 -> /DDR/DRAM_D15
- U2 pad A7: /DDR/DRAM_DQS1_P -> /DDR/DRAM_DQS1_N
- U2 pad A9: /DDR/NVCC_DRAM_1.2V -> /DDR/VDD_DRAM_1.2V
- U2 pad B1: /DDR/NVCC_DRAM_1.2V -> /DDR/VPP_2.5V
- U2 pad B3: /DDR/NVCC_DRAM_1.2V -> /DDR/VDD_DRAM_1.2V
- U2 pad B7: /DDR/DRAM_DQS1_N -> /DDR/DRAM_DQS1_P
- U2 pad B8: /DDR/DRAM_D09 -> /DDR/DRAM_D11
- U2 pad B9: /DDR/NVCC_DRAM_1.2V -> /DDR/VDD_DRAM_1.2V
- U2 pad C1: /DDR/NVCC_DRAM_1.2V -> /DDR/VDD_DRAM_1.2V
- U2 pad C2: /DDR/DRAM_D12 -> /DDR/DRAM_D14
- U2 pad C3: /DDR/DRAM_D10 -> /DDR/DRAM_D08
- U2 pad C7: /DDR/DRAM_D11 -> /DDR/DRAM_D10
- U2 pad C8: /DDR/DRAM_D13 -> /DDR/DRAM_D12
- U2 pad D1: /DDR/NVCC_DRAM_1.2V -> /DDR/VDD_DRAM_1.2V
- U2 pad D3: /DDR/DRAM_D14 -> /DDR/DRAM_D09
- U2 pad D7: /DDR/DRAM_D15 -> /DDR/DRAM_D13
- U2 pad D9: /DDR/NVCC_DRAM_1.2V -> /DDR/VDD_DRAM_1.2V
- U2 pad F2: /DDR/NVCC_DRAM_1.2V -> /DDR/VDD_DRAM_1.2V
- U2 pad F3: /DDR/DRAM_DQS0_P -> /DDR/DRAM_DQS0_N
- U2 pad F7: /DDR/DRAM_D01 -> /DDR/DRAM_D04
- U2 pad F8: /DDR/NVCC_DRAM_1.2V -> /DDR/VDD_DRAM_1.2V
- U2 pad G1: /DDR/NVCC_DRAM_1.2V -> /DDR/VDD_DRAM_1.2V
- U2 pad G3: /DDR/DRAM_DQS0_N -> /DDR/DRAM_DQS0_P
- U2 pad G7: /DDR/NVCC_DRAM_1.2V -> /DDR/VDD_DRAM_1.2V
- U2 pad G9: /DDR/NVCC_DRAM_1.2V -> /DDR/VDD_DRAM_1.2V
- U2 pad H2: /DDR/DRAM_D04 -> /DDR/DRAM_D01
- U2 pad H3: /DDR/DRAM_D02 -> /DDR/DRAM_D07
- U2 pad H7: /DDR/DRAM_D03 -> /DDR/DRAM_D02
- U2 pad H8: /DDR/DRAM_D05 -> /DDR/DRAM_D03
- U2 pad J1: /DDR/NVCC_DRAM_1.2V -> /DDR/VDD_DRAM_1.2V
- U2 pad J2: /DDR/NVCC_DRAM_1.2V -> /DDR/VDD_DRAM_1.2V
- U2 pad J7: /DDR/DRAM_D07 -> /DDR/DRAM_D05
- U2 pad J8: /DDR/NVCC_DRAM_1.2V -> /DDR/VDD_DRAM_1.2V
- U2 pad J9: /DDR/NVCC_DRAM_1.2V -> /DDR/VDD_DRAM_1.2V
- U2 pad L1: /DDR/NVCC_DRAM_1.2V -> /DDR/VDD_DRAM_1.2V
- U2 pad L9: /DDR/NVCC_DRAM_1.2V -> /DDR/VDD_DRAM_1.2V
- U2 pad R1: /DDR/NVCC_DRAM_1.2V -> /DDR/VDD_DRAM_1.2V
- U2 pad R9: /DDR/NVCC_DRAM_1.2V -> /DDR/VPP_2.5V
- U2 pad T9: /DDR/NVCC_DRAM_1.2V -> /DDR/VDD_DRAM_1.2V
- U20 pad B1: VDD -> VDD_3.3V
- U22 pad 10: VDD -> VDD_3.3V
- U22 pad 9: /USB/USB3_VBUS -> Net-(R48-Pad2)
- U29 pad 8: VCC -> VDD_1.8V
- U3 pad 1: VDD -> VDD_3.3V
- U3 pad 10: /Misc/CLK_32K_OUT -> /Misc/NVCC_SNVS_1.8V
- U3 pad 28: /Misc/CLK_32K_OUT -> /Misc/NVCC_SNVS_1.8V
- U3 pad 38: /DDR/NVCC_DRAM_1.2V -> /Power/NVCC_DRAM_1.2V
- U3 pad 43: VCC -> VDD_1.8V
- U3 pad 46: VDD -> VDD_3.3V
- U3 pad 54: VCC -> VDD_1.8V
- U3 pad 56: VCC -> VDD_1.8V
- U3 pad 7: VDD -> VDD_3.3V
- U30 pad 4: VDD -> VDD_3.3V
- U34 pad 1: VDD -> VDD_3.3V
- U34 pad 10: VDD -> VDD_3.3V
- U35 pad 5: VCC -> VDD_1.8V
- U36 pad 5: VCC -> VDD_1.8V
- U5 pad 5: VCC -> VDD_1.8V
- U6 pad 5: VCC -> VDD_1.8V
- U8 pad 12: VDD -> VDD_3.3V
- U8 pad 5: VDD -> VDD_3.3V
Routing:
- net GND: track 0.00 -> 40.6 mm, vias 0 -> 35
- net /DDR/DRAM_A08: track 0.00 -> 29.3 mm, vias 0 -> 2
- net /DDR/DRAM_A07: track 0.00 -> 29.0 mm, vias 0 -> 2
- net /DDR/DRAM_A06: track 0.00 -> 26.2 mm, vias 0 -> 2
- net /DDR/DRAM_A11: track 0.00 -> 26.1 mm, vias 0 -> 2
- net /DDR/VDD_DRAM_1.2V: track 0.00 -> 26.0 mm, vias 0 -> 20
- net /DDR/DRAM_D00: track 0.00 -> 25.5 mm, vias 0 -> 2
- net /DDR/DRAM_D01: track 0.00 -> 25.1 mm, vias 0 -> 2
- net /DDR/DRAM_A09: track 0.00 -> 23.5 mm, vias 0 -> 2
- net /DDR/DRAM_PARITY: track 0.00 -> 22.4 mm, vias 0 -> 2
- net /DDR/~{DRAM_RESET}: track 0.00 -> 22.3 mm, vias 0 -> 2
- net /DDR/DRAM_D07: track 0.00 -> 22.1 mm, vias 0 -> 2
- net /DDR/~{DRAM_ACT}: track 0.00 -> 21.5 mm, vias 0 -> 2
- net /DDR/DRAM_DQS0_P: track 0.00 -> 21.2 mm, vias 0 -> 2
- net /DDR/DRAM_D06: track 0.00 -> 20.8 mm, vias 0 -> 2
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- added copper zone on In4.Cu, net /DDR/VDD_DRAM_1.2V
- added copper zone on In3.Cu, net GND
