File: usb.kicad_sch (KiCad schematic)
At the start: 81 parts, among them J1 USB_C_Receptacle_USB2.0, J2 USB_C_Receptacle_USB2.0, J3 USB_C_Receptacle_USB2.0, J4 USB_C_Receptacle_USB2.0, U1 MIMX8MM6DVTLZAA, U10 D5V0H1B2LP, U11 D5V0H1B2LP, U12 TPD4EUSB30, U13 TPD4EUSB30, U14 74LVC1G07, U15 74LVC1G07, U16 D5V0H1B2LP, U17 CH343P, U18 TPD4EUSB30, U19 INA231, U20 D5V0H1B2LP, U21 TS3USB221E, U22 TPD4EUSB30, U4 74LVC1G04, U5 74LVC1G04, U6 NX5P3363, U7 TUSB320LAI, U8 NX5P3363, U9 TUSB320LAI

Commit message: add inital ddr tool version, lots of routing work
Parts:
- removed FB1, FB2, FB3, FB4: FerriteBead, Resistor_SMD:R_0603_1608Metric, symbol Device:FerriteBead
- added C?: 1uF, Capacitor_SMD:C_0402_1005Metric, symbol Device:C
- added D? (x2): D_Schottky, symbol Device:D_Schottky
- added R48: 0R, Resistor_SMD:R_0402_1005Metric, symbol Device:R
- added R49: 10K, Resistor_SMD:R_0402_1005Metric, symbol Device:R
- C119: renamed from C117; footprint Capacitor_SMD:C_0201_0603Metric -> qsbc:C_0201_0603Metric
- C120: renamed from C118; footprint Capacitor_SMD:C_0201_0603Metric -> qsbc:C_0201_0603Metric
- R29, R30, R33, R34, R35, R36: footprint Resistor_SMD:R_0201_0603Metric -> qsbc:R_0201_0603Metric
- TP24: renamed from TP23; footprint TestPoint:TestPoint_Pad_D1.5mm -> TestPoint:TestPoint_Pad_D1.0mm
- renumbered C107 to C109, C108 to C110, C109 to C111, C110 to C112, C111 to C113, C112 to C114, C113 to C115, C114 to C116, C115 to C117, C116 to C118, C119 to C121, C120 to C122, C121 to C123, C122 to C124, C123 to C125, C124 to C126, R48 to R50, R49 to R51, R50 to R52, U9 to U10, U10 to U11, U11 to U12, U12 to U13, U13 to U14, U14 to U15, U15 to U16, U16 to U17, U17 to U18, U18 to U19, U19 to U20, U20 to U21, U21 to U22, U22 to U23, U4 to U5, U5 to U6, U6 to U7, U7 to U8, U8 to U9
Connections:
- net GND: now also J1.S1 (SHIELD), J2.S1 (SHIELD), J3.S1 (SHIELD), J4.S1 (SHIELD), C?.2
- net USB3_VBUS: now also D?.2 (A), R48.1; no longer R50.1, U22.9 (S)
- net VDD_3.3V: now also R49.1; no longer C124.1, U18.3 (VDD5), U18.6 (V3), U18.9 (USB_VBUS)
- net VSYS_5V: now also D?.2 (A)
- new net: R48.2, R49.2, R50.1, U22.9 (S)
- new net CH343_V3: C124.1, U18.6 (V3)
- new net VDD_UART_5V: C?.1, D?.1 (K), D?.1 (K), U18.3 (VDD5), U18.9 (USB_VBUS)

Commit message: v2 of ddr flytimes tool, lots of routing work, sch fixes
Parts:
- removed U15, U16: 74LVC1G07, Package_TO_SOT_SMD:SOT-23-5, symbol 74xGxx:74LVC1G07
- removed U5, U6: 74LVC1G04, Package_TO_SOT_SMD:SOT-23-5, symbol 74xGxx:74LVC1G04
- added R21, R22: 10K, Resistor_SMD:R_0402_1005Metric, symbol Device:R
- added U14: 74LVC2G07, Package_TO_SOT_SMD:SOT-886, symbol 74xGxx:74LVC2G07
- added U5: 74LVC2G04, Package_TO_SOT_SMD:SOT-886, symbol 74xGxx:74LVC2G04
- C113, C114: footprint Capacitor_SMD:C_0603_1608Metric -> Capacitor_SMD:C_0402_1005Metric
- D1, D2: renamed from D?; footprint (none) -> Diode_SMD:D_SOD-523
- R36: renamed from R34; footprint qsbc:R_0201_0603Metric -> Resistor_SMD:R_0402_1005Metric
- gave numbers to parts that had none: 1
- renumbered C121 to C122, C122 to C123, C123 to C124, C124 to C125, C125 to C126, C126 to C127, D1 to D3, D2 to D4, R21 to R23, R22 to R24, R23 to R25, R24 to R26, R25 to R27, R26 to R28, R27 to R29, R28 to R30, R29 to R31, R30 to R32, R31 to R33, R32 to R34, R33 to R35, R35 to R37, R36 to R38, R37 to R39, R38 to R40, R39 to R41, R40 to R42, R41 to R43, R42 to R44, R43 to R45, R44 to R46, R45 to R47, R46 to R48, R47 to R49, R48 to R50, R49 to R51, R50 to R52, R51 to R53, R52 to R54, TP24 to TP23, U11 to U10, U12 to U11, U13 to U12, U14 to U13, U17 to U15, U18 to U16, U19 to U17, U20 to U18, U21 to U19, U22 to U20, U23 to U21, U7 to U6, U8 to U7, U9 to U8, U10 to U9
Connections:
- net GND: now also R21.2, R22.2, U14.2 (GND), U14.2 (GND), U5.2 (GND), U5.2 (GND)
- net USB1_CC1: now also U12.2 (D1-), U12.9; no longer U12.1 (D1+), U12.10
- net USB1_CC2: now also U12.1 (D1+), U12.10; no longer U12.2 (D1-), U12.9
- net USB1_DN: now also U12.5 (D2-), U12.6; no longer U12.4 (D2+), U12.7
- net USB1_DP: now also U12.4 (D2+), U12.7; no longer U12.5 (D2-), U12.6
- net USB1_ID: now also U5.1
- net USB1_VBUS_EN: now also R21.1
- net USB2_CC1: now also U13.2 (D1-), U13.9; no longer U13.1 (D1+), U13.10
- net USB2_CC2: now also U13.1 (D1+), U13.10; no longer U13.2 (D1-), U13.9
- net USB2_DN: now also U13.5 (D2-), U13.6; no longer U13.4 (D2+), U13.7
- net USB2_DP: now also U13.4 (D2+), U13.7; no longer U13.5 (D2-), U13.6
- net USB2_ID: now also U5.3
- net USB2_VBUS_EN: now also R22.1
- net VCC: now also U14.5 (VCC), U14.5 (VCC), U5.5 (VCC), U5.5 (VCC)
- net at R39.2, U16.4 (UART_TXD): now also U14.3
- net at D4.1 (K): now also U14.4
- net at R29.1: now also U5.6
- net at R30.1: now also U5.4
- net at R40.2, U16.5 (UART_RXD): now also U14.1
- net at D3.1 (K): now also U14.6

Commit message: more routing work, prepare to change to x32 lpddr4
Parts:
- removed C112: 0.1uF, Capacitor_SMD:C_0402_1005Metric, symbol Device:C
- C111: DNP DNP -> (none)
Connections:
- net CH343_V3: now also C127.1, R51.1, U20.10 (VCC)
- net GND: now also U16.17 (EPAD); no longer U16.1 (VDDIO)
- net VDD_3.3V: no longer C127.1, R51.1, U20.10 (VCC)
Changed lines of the file:
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@@
     (stroke (width 0) (type default) (color 0 0 0 0))
   )
-  (wire (pts (xy 111.76 383.54) (xy 111.76 386.08))
-    (stroke (width 0) (type default) (color 0 0 0 0))
-  )
   (wire (pts (xy 304.8 129.54) (xy 318.77 129.54))
     (stroke (width 0) (type default) (color 0 0 0 0))
@@
     (stroke (width 0) (type default) (color 0 0 0 0))
   )
-  (wire (pts (xy 100.33 373.38) (xy 111.76 373.38))
-    (stroke (width 0) (type default) (color 0 0 0 0))
-  )
   (wire (pts (xy 77.47 363.22) (xy 77.47 354.33))
     (stroke (width 0) (type default) (color 0 0 0 0))
@@
     (stroke (width 0) (type default) (color 0 0 0 0))
   )
-  (wire (pts (xy 111.76 373.38) (xy 111.76 375.92))
-    (stroke (width 0) (type default) (color 0 0 0 0))
-  )
   (wire (pts (xy 373.38 138.43) (xy 438.15 138.43))
     (stroke (width 0) (type default) (color 0 0 0 0))
@@
     (effects (font (size 1.27 1.27)) (justify left bottom))
   )
-  (label "VDD_3.3V" (at 415.29 123.19 0)
-    (effects (font (size 1.27 1.27)) (justify left bottom))
-  )
   (label "USB3_DN" (at 386.08 49.53 0)
     (effects (font (size 1.27 1.27)) (justify left bottom))
@@
     (effects (font (size 1.27 1.27)) (justify left bottom))
   )
-  (label "VDD_1.8V" (at 100.33 373.38 0)
-    (effects (font (size 1.27 1.27)) (justify left bottom))
-  )
   (label "USB1_VBUS" (at 215.9 52.07 180)
     (effects (font (size 1.27 1.27)) (justify right bottom))
@@
     (effects (font (size 1.27 1.27)) (justify left bottom))
   )
+  (label "CH343_V3" (at 449.58 106.68 0)
+    (effects (font (size 1.27 1.27)) (justify left bottom))
+  )
   (label "VSYS_5V" (at 298.45 81.28 0)
     (effects (font (size 1.27 1.27)) (justify left bottom))
@@
     (effects (font (size 1.27 1.27)) (justify left bottom))
   )
+  (label "CH343_V3" (at 415.29 123.19 0)
+    (effects (font (size 1.27 1.27)) (justify left bottom))
+  )
   (label "VDD_1.8V" (at 100.33 247.65 0)
     (effects (font (size 1.27 1.27)) (justify left bottom))
@@
     (effects (font (size 1.27 1.27)) (justify left bottom))
   )
-  (label "VDD_3.3V" (at 449.58 106.68 0)
-    (effects (font (size 1.27 1.27)) (justify left bottom))
-  )
   (label "~{USB1_INT}" (at 63.5 220.98 0)
     (effects (font (size 1.27 1.27)) (justify left bottom))
@@
     )
     (pin "1")
-    (pin "1")
     (pin "10")
     (pin "11")
@@
     (pin "15")
     (pin "16")
+    (pin "17")
     (pin "2")
     (pin "3")
@@
       (effects (font (size 0.762 0.762)))
     )
-    (property "DNP" "DNP" (id 5) (at 116.84 260.35 0))
     (pin "1")
     (pin "2")
@@
     (pin "D19")
   )
-  (symbol (lib_id "Device:C") (at 111.76 379.73 0) (unit 1)
-    (in_bom yes) (on_board yes)
-    (property "Reference" "C112" (id 0) (at 115.57 378.4599 0)
-      (effects (font (size 1.27 1.27)) (justify left))
-    )
-    (property "Value" "0.1uF" (id 1) (at 115.57 380.9999 0)
-      (effects (font (size 1.27 1.27)) (justify left))
-    )
-    (property "Footprint" "Capacitor_SMD:C_0402_1005Metric" (id 2) (at 112.7252 383.54 0)
-      (effects (font (size 1.27 1.27)) hide)
-    )
-    (property "Datasheet" "~" (id 3) (at 111.76 379.73 0)
-      (effects (font (size 1.27 1.27)) hide)
-    )
-    (property "Rating" "25V/20%" (id 4) (at 118.11 383.54 0)
-      (effects (font (size 0.762 0.762)))
-    )
-    (property "DNP" "DNP" (id 5) (at 116.84 386.08 0))
-    (pin "1")
-    (pin "2")
-  )
   (symbol (lib_id "Device:R") (at 55.88 374.65 180) (unit 1)
     (in_bom yes) (on_board yes)
@@
     (pin "2")
   )
-  (symbol (lib_id "power:GND") (at 111.76 386.08 0) (unit 1)
-    (in_bom yes) (on_board yes) (fields_autoplaced)
-    (property "Reference" "#PWR074" (id 0) (at 111.76 392.43 0)
-      (effects (font (size 1.27 1.27)) hide)
-    )
-    (property "Value" "GND" (id 1) (at 111.76 391.16 0))
-    (property "Footprint" "" (id 2) (at 111.76 386.08 0)
-      (effects (font (size 1.27 1.27)) hide)
-    )
-    (property "Datasheet" "" (id 3) (at 111.76 386.08 0)
-      (effects (font (size 1.27 1.27)) hide)
-    )
-    (pin "1")
-  )
   (symbol (lib_id "Device:R") (at 185.42 130.81 0) (unit 1)

Commit message: inital routing of ddr data bus, sch work
Parts:
- removed C122: 0.1uF, Capacitor_SMD:C_0402_1005Metric, symbol Device:C
- renumbered C115 to C100, C116 to C101, C117 to C102, C118 to C103, C119 to C104, C120 to C105, C121 to C106, C123 to C107, C124 to C108, C125 to C109, C126 to C110, C127 to C111, C109 to C95, C110 to C96, C111 to C97, C113 to C98, C114 to C99, R19 to R17, R20 to R18, R21 to R19, R22 to R20, R23 to R21, R24 to R22, R25 to R23, R26 to R24, R27 to R25, R28 to R26, R29 to R27, R30 to R28, R31 to R29, R32 to R30, R33 to R31, R34 to R32, R35 to R33, R36 to R34, R37 to R35, R38 to R36, R39 to R37, R40 to R38, R41 to R39, R42 to R40, R43 to R41, R44 to R42, R45 to R43, R46 to R44, R47 to R45, R48 to R46, R49 to R47, R50 to R48, R51 to R49, R52 to R50, R53 to R51, R54 to R52, TP23 to TP21, U11 to U10, U12 to U11, U13 to U12, U14 to U13, U15 to U14, U16 to U15, U17 to U16, U18 to U17, U19 to U18, U20 to U19, U21 to U20, U5 to U4, U6 to U5, U7 to U6, U8 to U7, U9 to U8, U10 to U9
Other:
- note added: "Keep UART USB interface Powered when VSYS disconnected"
