File: ethernet.kicad_sch (KiCad schematic)
At the start: 45 parts, among them J5 ARJM11D7-502-AB-EW2, U1 MIMX8MM6DVTLZAA, U21 RTL8211FD, U22 TPD4E02B04, U23 TPD4E02B04, Y2 25MHz

Commit message: change USB-UART conn, add new 0402 fp, more pcb work
Parts:
- C112, C113, C114, C115, C116, C117, C118, C119, C120, C121, C122, C123: footprint Capacitor_SMD:C_0402_1005Metric -> qsbc:C_0402_1005Metric
- R62, R63, R64, R65, R66, R67, R68, R69, R70, R71, R72, R73, R74, R75, R76: footprint Resistor_SMD:R_0402_1005Metric -> qsbc:R_0402_1005Metric
Changed lines of the file:
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@@
       (effects (font (size 1.27 1.27)) (justify left))
     )
-    (property "Footprint" "Capacitor_SMD:C_0402_1005Metric" (id 2) (at 199.0852 113.03 0)
+    (property "Footprint" "qsbc:C_0402_1005Metric" (id 2) (at 199.0852 113.03 0)
       (effects (font (size 1.27 1.27)) hide)
     )
@@
       (effects (font (size 1.27 1.27)) (justify left))
     )
-    (property "Footprint" "Resistor_SMD:R_0402_1005Metric" (id 2) (at 287.782 190.5 90)
+    (property "Footprint" "qsbc:R_0402_1005Metric" (id 2) (at 287.782 190.5 90)
       (effects (font (size 1.27 1.27)) hide)
     )
@@
       (effects (font (size 1.27 1.27)) (justify left))
     )
-    (property "Footprint" "Capacitor_SMD:C_0402_1005Metric" (id 2) (at 211.7852 46.99 0)
+    (property "Footprint" "qsbc:C_0402_1005Metric" (id 2) (at 211.7852 46.99 0)
       (effects (font (size 1.27 1.27)) hide)
     )
@@
       (effects (font (size 1.27 1.27)) (justify left))
     )
-    (property "Footprint" "Capacitor_SMD:C_0402_1005Metric" (id 2) (at 249.8852 156.21 0)
+    (property "Footprint" "qsbc:C_0402_1005Metric" (id 2) (at 249.8852 156.21 0)
       (effects (font (size 1.27 1.27)) hide)
     )
@@
       (effects (font (size 1.27 1.27)) (justify left))
     )
-    (property "Footprint" "Capacitor_SMD:C_0402_1005Metric" (id 2) (at 240.9952 234.95 0)
+    (property "Footprint" "qsbc:C_0402_1005Metric" (id 2) (at 240.9952 234.95 0)
       (effects (font (size 1.27 1.27)) hide)
     )
@@
       (effects (font (size 1.27 1.27)) (justify left))
     )
-    (property "Footprint" "Capacitor_SMD:C_0402_1005Metric" (id 2) (at 199.0852 69.85 0)
+    (property "Footprint" "qsbc:C_0402_1005Metric" (id 2) (at 199.0852 69.85 0)
       (effects (font (size 1.27 1.27)) hide)
     )
@@
       (effects (font (size 1.27 1.27)) (justify left))
     )
-    (property "Footprint" "Capacitor_SMD:C_0402_1005Metric" (id 2) (at 262.5852 156.21 0)
+    (property "Footprint" "qsbc:C_0402_1005Metric" (id 2) (at 262.5852 156.21 0)
       (effects (font (size 1.27 1.27)) hide)
     )
@@
     (property "Reference" "R65" (id 0) (at 161.29 31.75 90))
     (property "Value" "0R" (id 1) (at 161.29 34.29 90))
-    (property "Footprint" "Resistor_SMD:R_0402_1005Metric" (id 2) (at 161.29 38.608 90)
+    (property "Footprint" "qsbc:R_0402_1005Metric" (id 2) (at 161.29 38.608 90)
       (effects (font (size 1.27 1.27)) hide)
     )
@@
       (effects (font (size 1.27 1.27)) (justify left))
     )
-    (property "Footprint" "Resistor_SMD:R_0402_1005Metric" (id 2) (at 266.192 196.85 90)
+    (property "Footprint" "qsbc:R_0402_1005Metric" (id 2) (at 266.192 196.85 90)
       (effects (font (size 1.27 1.27)) hide)
     )
@@
       (effects (font (size 1.27 1.27)) (justify left))
     )
-    (property "Footprint" "Resistor_SMD:R_0402_1005Metric" (id 2) (at 287.782 175.26 90)
+    (property "Footprint" "qsbc:R_0402_1005Metric" (id 2) (at 287.782 175.26 90)
       (effects (font (size 1.27 1.27)) hide)
     )
@@
       (effects (font (size 1.27 1.27)) (justify left))
     )
-    (property "Footprint" "Resistor_SMD:R_0402_1005Metric" (id 2) (at 300.482 97.79 90)
+    (property "Footprint" "qsbc:R_0402_1005Metric" (id 2) (at 300.482 97.79 90)
       (effects (font (size 1.27 1.27)) hide)
     )
@@
       (effects (font (size 1.27 1.27)) (justify left))
     )
-    (property "Footprint" "Resistor_SMD:R_0402_1005Metric" (id 2) (at 267.462 175.26 90)
+    (property "Footprint" "qsbc:R_0402_1005Metric" (id 2) (at 267.462 175.26 90)
       (effects (font (size 1.27 1.27)) hide)
     )
@@
       (effects (font (size 1.27 1.27)) (justify left))
     )
-    (property "Footprint" "Capacitor_SMD:C_0402_1005Metric" (id 2) (at 199.0852 92.71 0)
+    (property "Footprint" "qsbc:C_0402_1005Metric" (id 2) (at 199.0852 92.71 0)
       (effects (font (size 1.27 1.27)) hide)
     )
@@
     (property "Reference" "R68" (id 0) (at 161.29 97.79 90))
     (property "Value" "0R" (id 1) (at 161.29 100.33 90))
-    (property "Footprint" "Resistor_SMD:R_0402_1005Metric" (id 2) (at 161.29 104.648 90)
+    (property "Footprint" "qsbc:R_0402_1005Metric" (id 2) (at 161.29 104.648 90)
       (effects (font (size 1.27 1.27)) hide)
     )
@@
       (effects (font (size 1.27 1.27)) (justify left))
     )
-    (property "Footprint" "Resistor_SMD:R_0402_1005Metric" (id 2) (at 303.022 115.57 90)
+    (property "Footprint" "qsbc:R_0402_1005Metric" (id 2) (at 303.022 115.57 90)
       (effects (font (size 1.27 1.27)) hide)
     )
@@
       (effects (font (size 1.27 1.27)) (justify left))
     )
-    (property "Footprint" "Resistor_SMD:R_0402_1005Metric" (id 2) (at 111.252 204.47 90)
+    (property "Footprint" "qsbc:R_0402_1005Metric" (id 2) (at 111.252 204.47 90)
       (effects (font (size 1.27 1.27)) hide)
     )
@@
       (effects (font (size 1.27 1.27)) (justify left))
     )
-    (property "Footprint" "Capacitor_SMD:C_0402_1005Metric" (id 2) (at 224.4852 113.03 0)
+    (property "Footprint" "qsbc:C_0402_1005Metric" (id 2) (at 224.4852 113.03 0)
       (effects (font (size 1.27 1.27)) hide)
     )
@@
       (effects (font (size 1.27 1.27)) (justify left))
     )
-    (property "Footprint" "Resistor_SMD:R_0402_1005Metric" (id 2) (at 277.622 190.5 90)
+    (property "Footprint" "qsbc:R_0402_1005Metric" (id 2) (at 277.622 190.5 90)
       (effects (font (size 1.27 1.27)) hide)
     )
@@
       (effects (font (size 1.27 1.27)) (justify left))
     )
-    (property "Footprint" "Capacitor_SMD:C_0402_1005Metric" (id 2) (at 211.7852 113.03 0)
+    (property "Footprint" "qsbc:C_0402_1005Metric" (id 2) (at 211.7852 113.03 0)
       (effects (font (size 1.27 1.27)) hide)
     )
@@
     (property "Reference" "R66" (id 0) (at 161.29 54.61 90))
     (property "Value" "0R" (id 1) (at 161.29 57.15 90))
-    (property "Footprint" "Resistor_SMD:R_0402_1005Metric" (id 2) (at 161.29 61.468 90)
+    (property "Footprint" "qsbc:R_0402_1005Metric" (id 2) (at 161.29 61.468 90)
       (effects (font (size 1.27 1.27)) hide)
     )
@@
       (effects (font (size 1.27 1.27)) (justify left))
     )
-    (property "Footprint" "Resistor_SMD:R_0402_1005Metric" (id 2) (at 121.412 204.47 90)
+    (property "Footprint" "qsbc:R_0402_1005Metric" (id 2) (at 121.412 204.47 90)
       (effects (font (size 1.27 1.27)) hide)
     )
@@
       (effects (font (size 1.27 1.27)) (justify left))
     )
-    (property "Footprint" "Capacitor_SMD:C_0402_1005Metric" (id 2) (at 211.7852 69.85 0)
+    (property "Footprint" "qsbc:C_0402_1005Metric" (id 2) (at 211.7852 69.85 0)
       (effects (font (size 1.27 1.27)) hide)
     )
@@
       (effects (font (size 1.27 1.27)) (justify left))
     )
-    (property "Footprint" "Capacitor_SMD:C_0402_1005Metric" (id 2) (at 199.0852 46.99 0)
+    (property "Footprint" "qsbc:C_0402_1005Metric" (id 2) (at 199.0852 46.99 0)
       (effects (font (size 1.27 1.27)) hide)
     )
@@
       (effects (font (size 1.27 1.27)) (justify left))
     )
-    (property "Footprint" "Resistor_SMD:R_0402_1005Metric" (id 2) (at 143.002 204.47 90)
+    (property "Footprint" "qsbc:R_0402_1005Metric" (id 2) (at 143.002 204.47 90)
       (effects (font (size 1.27 1.27)) hide)
     )
@@
       (effects (font (size 1.27 1.27)) (justify left))
     )
-    (property "Footprint" "Capacitor_SMD:C_0402_1005Metric" (id 2) (at 253.6952 234.95 0)
+    (property "Footprint" "qsbc:C_0402_1005Metric" (id 2) (at 253.6952 234.95 0)
       (effects (font (size 1.27 1.27)) hide)
     )
@@
     (property "Reference" "R67" (id 0) (at 161.29 77.47 90))
     (property "Value" "0R" (id 1) (at 161.29 80.01 90))
-    (property "Footprint" "Resistor_SMD:R_0402_1005Metric" (id 2) (at 161.29 84.328 90)
+    (property "Footprint" "qsbc:R_0402_1005Metric" (id 2) (at 161.29 84.328 90)
       (effects (font (size 1.27 1.27)) hide)
     )
@@
       (effects (font (size 1.27 1.27)) (justify left))
     )
-    (property "Footprint" "Resistor_SMD:R_0402_1005Metric" (id 2) (at 259.842 135.89 90)
-      (effects (font (size 1.27 1.27)) hide)
-    )
+    (property "Footprint" "qsbc:R_0402_1005Metric" (id 2) (at 259.842 135.89 90)
+      (effects (font (size 1.27 1.27)) hide)
+    )

Commit message: pmic routing almost done
Parts:
- C124: footprint Capacitor_SMD:C_0603_1608Metric -> qsbc:C_0603_1608Metric
Changed lines of the file:
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@@
       (effects (font (size 1.27 1.27)) (justify left))
     )
-    (property "Footprint" "Capacitor_SMD:C_0603_1608Metric" (id 2) (at 300.6852 76.2 0)
+    (property "Footprint" "qsbc:C_0603_1608Metric" (id 2) (at 300.6852 76.2 0)
       (effects (font (size 1.27 1.27)) hide)
     )
