File: ddr_power.kicad_sch (KiCad schematic)
At the start: 27 parts, among them U2 MT53D512M32D2DS

Commit message: bom work, change uart level shifter and m.2 socket
Parts:
- C161, C162, C163, C164, C165, C166, C167, C168, C169, C170, C171, C172: MPN (none) -> GRM155R60J106ME44D
- C173, C174, C175, C176, C177, C178, C179, C180, C181, C182, C183, C184, C185, C186: MPN (none) -> GRM033R60J224ME15D
- U2: MPN (none) -> MT53D512M32D2DS-053WT:D
Changed lines of the file:
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@@
       (effects (font (size 0.762 0.762)))
+    )
+    (property "MPN" "GRM155R60J106ME44D" (id 5) (at 120.65 59.69 0)
+      (effects (font (size 1.27 1.27)) hide)
     )
     (pin "1")
@@
       (effects (font (size 0.762 0.762)))
     )
+    (property "MPN" "GRM033R60J224ME15D" (id 5) (at 190.5 59.69 0)
+      (effects (font (size 1.27 1.27)) hide)
+    )
     (pin "1")
     (pin "2")
@@
       (effects (font (size 0.762 0.762)))
     )
+    (property "MPN" "GRM033R60J224ME15D" (id 5) (at 162.56 97.79 0)
+      (effects (font (size 1.27 1.27)) hide)
+    )
     (pin "1")
     (pin "2")
@@
     (property "Rating" "6.3V/20%" (id 4) (at 196.85 180.34 0)
       (effects (font (size 0.762 0.762)))
+    )
+    (property "MPN" "GRM033R60J224ME15D" (id 5) (at 190.5 176.53 0)
+      (effects (font (size 1.27 1.27)) hide)
     )
     (pin "1")
@@
     )
     (property "Datasheet" "https://media-www.micron.com/-/media/client/global/documents/products/data-sheet/dram/mobile-dram/low-power-dram/lpddr4/200b_z11m_non_auto_lpddr4_lpddr4x.pdf?rev=3a9658f2622d43c4ae5713671b1e9e43" (id 3) (at 250.19 240.03 0)
+      (effects (font (size 1.27 1.27)) hide)
+    )
+    (property "MPN" "MT53D512M32D2DS-053WT:D" (id 4) (at 250.19 125.73 0)
       (effects (font (size 1.27 1.27)) hide)
     )
@@
       (effects (font (size 0.762 0.762)))
     )
+    (property "MPN" "GRM155R60J106ME44D" (id 5) (at 148.59 59.69 0)
+      (effects (font (size 1.27 1.27)) hide)
+    )
     (pin "1")
     (pin "2")
@@
       (effects (font (size 0.762 0.762)))
     )
+    (property "MPN" "GRM033R60J224ME15D" (id 5) (at 190.5 97.79 0)
+      (effects (font (size 1.27 1.27)) hide)
+    )
     (pin "1")
     (pin "2")
@@
     (property "Rating" "6.3V/20%" (id 4) (at 182.88 63.5 0)
       (effects (font (size 0.762 0.762)))
+    )
+    (property "MPN" "GRM033R60J224ME15D" (id 5) (at 176.53 59.69 0)
+      (effects (font (size 1.27 1.27)) hide)
     )
     (pin "1")
@@
       (effects (font (size 0.762 0.762)))
     )
+    (property "MPN" "GRM155R60J106ME44D" (id 5) (at 134.62 59.69 0)
+      (effects (font (size 1.27 1.27)) hide)
+    )
     (pin "1")
     (pin "2")
@@
       (effects (font (size 0.762 0.762)))
     )
+    (property "MPN" "GRM033R60J224ME15D" (id 5) (at 204.47 176.53 0)
+      (effects (font (size 1.27 1.27)) hide)
+    )
     (pin "1")
     (pin "2")
@@
       (effects (font (size 0.762 0.762)))
     )
+    (property "MPN" "GRM155R60J106ME44D" (id 5) (at 92.71 176.53 0)
+      (effects (font (size 1.27 1.27)) hide)
+    )
     (pin "1")
     (pin "2")
@@
       (effects (font (size 0.762 0.762)))
     )
+    (property "MPN" "GRM033R60J224ME15D" (id 5) (at 204.47 97.79 0)
+      (effects (font (size 1.27 1.27)) hide)
+    )
     (pin "1")
     (pin "2")
@@
       (effects (font (size 0.762 0.762)))
     )
+    (property "MPN" "GRM033R60J224ME15D" (id 5) (at 204.47 59.69 0)
+      (effects (font (size 1.27 1.27)) hide)
+    )
     (pin "1")
     (pin "2")
@@
       (effects (font (size 0.762 0.762)))
     )
+    (property "MPN" "GRM155R60J106ME44D" (id 5) (at 120.65 97.79 0)
+      (effects (font (size 1.27 1.27)) hide)
+    )
     (pin "1")
     (pin "2")
@@
     (property "Rating" "6.3V/20%" (id 4) (at 182.88 180.34 0)
       (effects (font (size 0.762 0.762)))
+    )
+    (property "MPN" "GRM033R60J224ME15D" (id 5) (at 176.53 176.53 0)
+      (effects (font (size 1.27 1.27)) hide)
     )
     (pin "1")
@@
       (effects (font (size 0.762 0.762)))
     )
+    (property "MPN" "GRM033R60J224ME15D" (id 5) (at 162.56 59.69 0)
+      (effects (font (size 1.27 1.27)) hide)
+    )
     (pin "1")
     (pin "2")
@@
       (effects (font (size 0.762 0.762)))
     )
+    (property "MPN" "GRM033R60J224ME15D" (id 5) (at 148.59 97.79 0)
+      (effects (font (size 1.27 1.27)) hide)
+    )
     (pin "1")
     (pin "2")
@@
     (property "Rating" "6.3V/20%" (id 4) (at 113.03 63.5 0)
       (effects (font (size 0.762 0.762)))
+    )
+    (property "MPN" "GRM155R60J106ME44D" (id 5) (at 106.68 59.69 0)
+      (effects (font (size 1.27 1.27)) hide)
     )
     (pin "1")
@@
       (effects (font (size 0.762 0.762)))
     )
+    (property "MPN" "GRM155R60J106ME44D" (id 5) (at 106.68 176.53 0)
+      (effects (font (size 1.27 1.27)) hide)
+    )
     (pin "1")
     (pin "2")
@@
       (effects (font (size 0.762 0.762)))
     )
+    (property "MPN" "GRM155R60J106ME44D" (id 5) (at 134.62 176.53 0)
+      (effects (font (size 1.27 1.27)) hide)
+    )
     (pin "1")
     (pin "2")
@@
       (effects (font (size 0.762 0.762)))
     )
+    (property "MPN" "GRM033R60J224ME15D" (id 5) (at 148.59 176.53 0)
+      (effects (font (size 1.27 1.27)) hide)
+    )
     (pin "1")
     (pin "2")
@@
       (effects (font (size 0.762 0.762)))
     )
+    (property "MPN" "GRM155R60J106ME44D" (id 5) (at 134.62 97.79 0)
+      (effects (font (size 1.27 1.27)) hide)
+    )
     (pin "1")
     (pin "2")
@@
       (effects (font (size 0.762 0.762)))
     )
+    (property "MPN" "GRM155R60J106ME44D" (id 5) (at 106.68 97.79 0)
+      (effects (font (size 1.27 1.27)) hide)
+    )
     (pin "1")
     (pin "2")
@@
       (effects (font (size 0.762 0.762)))
     )
+    (property "MPN" "GRM033R60J224ME15D" (id 5) (at 162.56 176.53 0)
+      (effects (font (size 1.27 1.27)) hide)
+    )
     (pin "1")
     (pin "2")
@@
       (effects (font (size 0.762 0.762)))
     )
+    (property "MPN" "GRM155R60J106ME44D" (id 5) (at 120.65 176.53 0)
+      (effects (font (size 1.27 1.27)) hide)
+    )
     (pin "1")
     (pin "2")
@@
       (effects (font (size 0.762 0.762)))
     )
+    (property "MPN" "GRM033R60J224ME15D" (id 5) (at 176.53 97.79 0)
+      (effects (font (size 1.27 1.27)) hide)
+    )
     (pin "1")
     (pin "2")
@@
       (effects (font (size 0.762 0.762)))
     )
-    (pin "1")
+    (property "MPN" "GRM155R60J106ME44D" (id 5) (at 92.71 97.79 0)
+      (effects (font (size 1.27 1.27)) hide)
+    )
+    (pin "1")
