File: pcie.kicad_sch (KiCad schematic)
At the start: 28 parts, among them J10 1-2199119-6, U1 MIMX8MM6DVTLZAA, U34 SI52112-B5-GM2, U35 74LVC2G07, Y4 25MHz

Commit message: Rev 1
Parts:
- renumbered R134 to R133, R135 to R134, R136 to R135, R137 to R136, R138 to R137, R139 to R138, R140 to R139, R141 to R140
Connections:
- net PCIE_REFCLK_N: now also U1.A21 (PCIE_CLK_N); no longer U1.B21 (PCIE_CLK_P)
- net PCIE_REFCLK_P: now also U1.B21 (PCIE_CLK_P); no longer U1.A21 (PCIE_CLK_N)
- net PCIE_TX_R_N: now also C155.2, J10.47 (PETn0/SATA-A-); no longer C154.2, J10.49 (PETp0/SATA-A+)
- net PCIE_TX_R_P: now also C154.2, J10.49 (PETp0/SATA-A+); no longer C155.2, J10.47 (PETn0/SATA-A-)
Other:
- note added: "P/N swap for routing"
Changed lines of the file:
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@@
   (title_block
     (title "QSBC")
-    (rev "1")
+    (date "2022-12-01")
+    (rev "1.0")
     (company "Q-LAB")
   )
@@
     (effects (font (size 1.27 1.27)) (justify left bottom))
   )
+  (text "P/N swap for routing" (at 142.24 91.44 0)
+    (effects (font (size 1.27 1.27)) (justify left bottom))
+  )
   (label "~{M2_WAKE_3.3V}" (at 193.04 66.04 0)
     (effects (font (size 1.27 1.27)) (justify left bottom))
@@
     (effects (font (size 1.27 1.27)) (justify left bottom))
   )
-  (label "PCIE_REFCLK_N" (at 105.41 62.23 0)
-    (effects (font (size 1.27 1.27)) (justify left bottom))
-  )
-  (label "PCIE_TX_R_P" (at 193.04 73.66 0)
+  (label "PCIE_REFCLK_N" (at 105.41 59.69 0)
+    (effects (font (size 1.27 1.27)) (justify left bottom))
+  )
+  (label "PCIE_TX_R_P" (at 193.04 71.12 0)
     (effects (font (size 1.27 1.27)) (justify left bottom))
   )
@@
     (effects (font (size 1.27 1.27)) (justify left bottom))
   )
-  (label "PCIE_REFCLK_P" (at 105.41 59.69 0)
+  (label "PCIE_REFCLK_P" (at 105.41 62.23 0)
     (effects (font (size 1.27 1.27)) (justify left bottom))
   )
@@
     (effects (font (size 1.27 1.27)) (justify right bottom))
   )
-  (label "PCIE_TX_R_N" (at 193.04 71.12 0)
+  (label "PCIE_TX_R_N" (at 193.04 73.66 0)
     (effects (font (size 1.27 1.27)) (justify left bottom))
   )
@@
   (symbol (lib_id "power:GND") (at 236.22 154.94 0) (unit 1)
     (in_bom yes) (on_board yes) (fields_autoplaced)
-    (property "Reference" "#PWR0155" (id 0) (at 236.22 161.29 0)
+    (property "Reference" "#PWR0154" (id 0) (at 236.22 161.29 0)
       (effects (font (size 1.27 1.27)) hide)
     )
@@
   (symbol (lib_id "Device:R") (at 266.7 97.79 0) (unit 1)
     (in_bom yes) (on_board yes)
-    (property "Reference" "R138" (id 0) (at 269.24 96.5199 0)
+    (property "Reference" "R137" (id 0) (at 269.24 96.5199 0)
       (effects (font (size 1.27 1.27)) (justify left))
     )
@@
   (symbol (lib_id "power:GND") (at 119.38 153.67 0) (unit 1)
     (in_bom yes) (on_board yes) (fields_autoplaced)
-    (property "Reference" "#PWR0151" (id 0) (at 119.38 160.02 0)
+    (property "Reference" "#PWR0150" (id 0) (at 119.38 160.02 0)
       (effects (font (size 1.27 1.27)) hide)
     )
@@
   (symbol (lib_id "power:GND") (at 266.7 39.37 0) (unit 1)
     (in_bom yes) (on_board yes) (fields_autoplaced)
-    (property "Reference" "#PWR0156" (id 0) (at 266.7 45.72 0)
+    (property "Reference" "#PWR0155" (id 0) (at 266.7 45.72 0)
       (effects (font (size 1.27 1.27)) hide)
     )
@@
   (symbol (lib_id "power:GND") (at 121.92 91.44 0) (unit 1)
     (in_bom yes) (on_board yes) (fields_autoplaced)
-    (property "Reference" "#PWR0152" (id 0) (at 121.92 97.79 0)
+    (property "Reference" "#PWR0151" (id 0) (at 121.92 97.79 0)
       (effects (font (size 1.27 1.27)) hide)
     )
@@
   (symbol (lib_id "Device:R") (at 121.92 85.09 0) (unit 1)
     (in_bom yes) (on_board yes)
-    (property "Reference" "R134" (id 0) (at 124.46 83.8199 0)
+    (property "Reference" "R133" (id 0) (at 124.46 83.8199 0)
       (effects (font (size 1.27 1.27)) (justify left))
     )
@@
   (symbol (lib_id "Device:R") (at 340.36 54.61 0) (unit 1)
     (in_bom yes) (on_board yes)
-    (property "Reference" "R140" (id 0) (at 342.9 53.3399 0)
+    (property "Reference" "R139" (id 0) (at 342.9 53.3399 0)
       (effects (font (size 1.27 1.27)) (justify left))
     )
@@
   (symbol (lib_id "Device:R") (at 172.72 54.61 0) (unit 1)
     (in_bom yes) (on_board yes)
-    (property "Reference" "R136" (id 0) (at 175.26 53.3399 0)
+    (property "Reference" "R135" (id 0) (at 175.26 53.3399 0)
       (effects (font (size 1.27 1.27)) (justify left))
     )
@@
   (symbol (lib_id "Device:R") (at 285.75 118.11 0) (unit 1)
     (in_bom yes) (on_board yes)
-    (property "Reference" "R139" (id 0) (at 288.29 116.8399 0)
+    (property "Reference" "R138" (id 0) (at 288.29 116.8399 0)
       (effects (font (size 1.27 1.27)) (justify left))
     )
@@
   (symbol (lib_id "Device:R") (at 182.88 54.61 0) (unit 1)
     (in_bom yes) (on_board yes)
-    (property "Reference" "R137" (id 0) (at 185.42 53.3399 0)
+    (property "Reference" "R136" (id 0) (at 185.42 53.3399 0)
       (effects (font (size 1.27 1.27)) (justify left))
     )
@@
   (symbol (lib_id "power:GND") (at 90.17 133.35 0) (unit 1)
     (in_bom yes) (on_board yes) (fields_autoplaced)
-    (property "Reference" "#PWR0150" (id 0) (at 90.17 139.7 0)
+    (property "Reference" "#PWR0149" (id 0) (at 90.17 139.7 0)
       (effects (font (size 1.27 1.27)) hide)
     )
@@
   (symbol (lib_id "power:GND") (at 361.95 106.68 0) (unit 1)
     (in_bom yes) (on_board yes) (fields_autoplaced)
-    (property "Reference" "#PWR0157" (id 0) (at 361.95 113.03 0)
+    (property "Reference" "#PWR0156" (id 0) (at 361.95 113.03 0)
       (effects (font (size 1.27 1.27)) hide)
     )
@@
   (symbol (lib_id "power:GND") (at 363.22 66.04 0) (unit 1)
     (in_bom yes) (on_board yes) (fields_autoplaced)
-    (property "Reference" "#PWR0158" (id 0) (at 363.22 72.39 0)
+    (property "Reference" "#PWR0157" (id 0) (at 363.22 72.39 0)
       (effects (font (size 1.27 1.27)) hide)
     )
@@
   (symbol (lib_id "power:GND") (at 381 49.53 0) (unit 1)
     (in_bom yes) (on_board yes) (fields_autoplaced)
-    (property "Reference" "#PWR0159" (id 0) (at 381 55.88 0)
+    (property "Reference" "#PWR0158" (id 0) (at 381 55.88 0)
       (effects (font (size 1.27 1.27)) hide)
     )
@@
   (symbol (lib_id "Device:R") (at 162.56 54.61 0) (unit 1)
     (in_bom yes) (on_board yes)
-    (property "Reference" "R135" (id 0) (at 165.1 53.3399 0)
+    (property "Reference" "R134" (id 0) (at 165.1 53.3399 0)
       (effects (font (size 1.27 1.27)) (justify left))
     )
@@
   (symbol (lib_id "power:GND") (at 132.08 139.7 0) (unit 1)
     (in_bom yes) (on_board yes) (fields_autoplaced)
-    (property "Reference" "#PWR0153" (id 0) (at 132.08 146.05 0)
+    (property "Reference" "#PWR0152" (id 0) (at 132.08 146.05 0)
       (effects (font (size 1.27 1.27)) hide)
     )
@@
   (symbol (lib_id "power:GND") (at 176.53 109.22 0) (unit 1)
     (in_bom yes) (on_board yes) (fields_autoplaced)
-    (property "Reference" "#PWR0154" (id 0) (at 176.53 115.57 0)
+    (property "Reference" "#PWR0153" (id 0) (at 176.53 115.57 0)
       (effects (font (size 1.27 1.27)) hide)
     )
@@
   (symbol (lib_id "Device:R") (at 340.36 95.25 0) (unit 1)
     (in_bom yes) (on_board yes)
-    (property "Reference" "R141" (id 0) (at 342.9 93.9799 0)
-      (effects (font (size 1.27 1.27)) (justify left))
-    )
+    (property "Reference" "R140" (id 0) (at 342.9 93.9799 0)
+      (effects (font (size 1.27 1.27)) (justify left))
+    )
