File: power.kicad_sch (KiCad schematic)
At the start: 71 parts, among them SW1 SW_Push, U3 BD71847MWV, Y1 Crystal

Commit message: change USB-UART conn, add new 0402 fp, more pcb work
Parts:
- C58, C59, C60, C61, C62, C63, C72, C73, C74, C75, C76, C77, C90, C92, C93, C94: footprint Capacitor_SMD:C_0402_1005Metric -> qsbc:C_0402_1005Metric
- R11, R12, R13, R14, R15, R16: footprint Resistor_SMD:R_0402_1005Metric -> qsbc:R_0402_1005Metric
Changed lines of the file:
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@@
       (effects (font (size 1.27 1.27)) (justify left))
     )
-    (property "Footprint" "Capacitor_SMD:C_0402_1005Metric" (id 2) (at 351.4852 284.48 0)
+    (property "Footprint" "qsbc:C_0402_1005Metric" (id 2) (at 351.4852 284.48 0)
       (effects (font (size 1.27 1.27)) hide)
     )
@@
       (effects (font (size 1.27 1.27)) (justify left))
     )
-    (property "Footprint" "Capacitor_SMD:C_0402_1005Metric" (id 2) (at 84.7852 330.2 0)
+    (property "Footprint" "qsbc:C_0402_1005Metric" (id 2) (at 84.7852 330.2 0)
       (effects (font (size 1.27 1.27)) hide)
     )
@@
       (effects (font (size 1.27 1.27)) (justify left))
     )
-    (property "Footprint" "Capacitor_SMD:C_0402_1005Metric" (id 2) (at 195.2752 255.27 0)
+    (property "Footprint" "qsbc:C_0402_1005Metric" (id 2) (at 195.2752 255.27 0)
       (effects (font (size 1.27 1.27)) hide)
     )
@@
       (effects (font (size 1.27 1.27)) (justify left))
     )
-    (property "Footprint" "Resistor_SMD:R_0402_1005Metric" (id 2) (at 319.532 237.49 90)
+    (property "Footprint" "qsbc:R_0402_1005Metric" (id 2) (at 319.532 237.49 90)
       (effects (font (size 1.27 1.27)) hide)
     )
@@
       (effects (font (size 1.27 1.27)) (justify left))
     )
-    (property "Footprint" "Capacitor_SMD:C_0402_1005Metric" (id 2) (at 72.0852 203.2 0)
+    (property "Footprint" "qsbc:C_0402_1005Metric" (id 2) (at 72.0852 203.2 0)
       (effects (font (size 1.27 1.27)) hide)
     )
@@
       (effects (font (size 1.27 1.27)) (justify left))
     )
-    (property "Footprint" "Capacitor_SMD:C_0402_1005Metric" (id 2) (at 59.3852 203.2 0)
+    (property "Footprint" "qsbc:C_0402_1005Metric" (id 2) (at 59.3852 203.2 0)
       (effects (font (size 1.27 1.27)) hide)
     )
@@
       (effects (font (size 1.27 1.27)) (justify left))
     )
-    (property "Footprint" "Capacitor_SMD:C_0402_1005Metric" (id 2) (at 331.1652 284.48 0)
+    (property "Footprint" "qsbc:C_0402_1005Metric" (id 2) (at 331.1652 284.48 0)
       (effects (font (size 1.27 1.27)) hide)
     )
@@
       (effects (font (size 1.27 1.27)) (justify left))
     )
-    (property "Footprint" "Capacitor_SMD:C_0402_1005Metric" (id 2) (at 194.0052 201.93 0)
+    (property "Footprint" "qsbc:C_0402_1005Metric" (id 2) (at 194.0052 201.93 0)
       (effects (font (size 1.27 1.27)) hide)
     )
@@
       (effects (font (size 1.27 1.27)) (justify left))
     )
-    (property "Footprint" "Capacitor_SMD:C_0402_1005Metric" (id 2) (at 195.2752 237.49 0)
+    (property "Footprint" "qsbc:C_0402_1005Metric" (id 2) (at 195.2752 237.49 0)
       (effects (font (size 1.27 1.27)) hide)
     )
@@
       (effects (font (size 1.27 1.27)) (justify left))
     )
-    (property "Footprint" "Capacitor_SMD:C_0402_1005Metric" (id 2) (at 195.2752 293.37 0)
+    (property "Footprint" "qsbc:C_0402_1005Metric" (id 2) (at 195.2752 293.37 0)
       (effects (font (size 1.27 1.27)) hide)
     )
@@
       (effects (font (size 1.27 1.27)) (justify left))
     )
-    (property "Footprint" "Capacitor_SMD:C_0402_1005Metric" (id 2) (at 84.7852 274.32 0)
+    (property "Footprint" "qsbc:C_0402_1005Metric" (id 2) (at 84.7852 274.32 0)
       (effects (font (size 1.27 1.27)) hide)
     )
@@
     (property "Reference" "R12" (id 0) (at 340.36 250.19 90))
     (property "Value" "1M" (id 1) (at 340.36 252.73 90))
-    (property "Footprint" "Resistor_SMD:R_0402_1005Metric" (id 2) (at 340.36 258.318 90)
+    (property "Footprint" "qsbc:R_0402_1005Metric" (id 2) (at 340.36 258.318 90)
       (effects (font (size 1.27 1.27)) hide)
     )
@@
       (effects (font (size 1.27 1.27)) (justify left))
     )
-    (property "Footprint" "Capacitor_SMD:C_0402_1005Metric" (id 2) (at 194.0052 219.71 0)
+    (property "Footprint" "qsbc:C_0402_1005Metric" (id 2) (at 194.0052 219.71 0)
       (effects (font (size 1.27 1.27)) hide)
     )
@@
       (effects (font (size 1.27 1.27)) (justify left))
     )
-    (property "Footprint" "Resistor_SMD:R_0402_1005Metric" (id 2) (at 346.202 210.82 90)
+    (property "Footprint" "qsbc:R_0402_1005Metric" (id 2) (at 346.202 210.82 90)
       (effects (font (size 1.27 1.27)) hide)
     )
@@
       (effects (font (size 1.27 1.27)) (justify left))
     )
-    (property "Footprint" "Capacitor_SMD:C_0402_1005Metric" (id 2) (at 84.7852 238.76 0)
+    (property "Footprint" "qsbc:C_0402_1005Metric" (id 2) (at 84.7852 238.76 0)
       (effects (font (size 1.27 1.27)) hide)
     )
@@
       (effects (font (size 1.27 1.27)) (justify left))
     )
-    (property "Footprint" "Capacitor_SMD:C_0402_1005Metric" (id 2) (at 84.7852 203.2 0)
+    (property "Footprint" "qsbc:C_0402_1005Metric" (id 2) (at 84.7852 203.2 0)
       (effects (font (size 1.27 1.27)) hide)
     )
@@
     (property "Reference" "R13" (id 0) (at 341.63 148.59 90))
     (property "Value" "0R" (id 1) (at 341.63 151.13 90))
-    (property "Footprint" "Resistor_SMD:R_0402_1005Metric" (id 2) (at 341.63 156.718 90)
+    (property "Footprint" "qsbc:R_0402_1005Metric" (id 2) (at 341.63 156.718 90)
       (effects (font (size 1.27 1.27)) hide)
     )
@@
       (effects (font (size 1.27 1.27)) (justify left))
     )
-    (property "Footprint" "Resistor_SMD:R_0402_1005Metric" (id 2) (at 356.362 210.82 90)
+    (property "Footprint" "qsbc:R_0402_1005Metric" (id 2) (at 356.362 210.82 90)
       (effects (font (size 1.27 1.27)) hide)
     )
@@
       (effects (font (size 1.27 1.27)) (justify left))
     )
-    (property "Footprint" "Capacitor_SMD:C_0402_1005Metric" (id 2) (at 371.8052 204.47 0)
+    (property "Footprint" "qsbc:C_0402_1005Metric" (id 2) (at 371.8052 204.47 0)
       (effects (font (size 1.27 1.27)) hide)
     )
@@
       (effects (font (size 1.27 1.27)) (justify left))
     )
-    (property "Footprint" "Capacitor_SMD:C_0402_1005Metric" (id 2) (at 195.2752 273.05 0)
+    (property "Footprint" "qsbc:C_0402_1005Metric" (id 2) (at 195.2752 273.05 0)
       (effects (font (size 1.27 1.27)) hide)
     )
@@
     (property "Reference" "R14" (id 0) (at 341.63 158.75 90))
     (property "Value" "0R" (id 1) (at 341.63 161.29 90))
-    (property "Footprint" "Resistor_SMD:R_0402_1005Metric" (id 2) (at 341.63 166.878 90)
+    (property "Footprint" "qsbc:R_0402_1005Metric" (id 2) (at 341.63 166.878 90)
       (effects (font (size 1.27 1.27)) hide)
     )
@@
       (effects (font (size 1.27 1.27)) (justify left))
     )
-    (property "Footprint" "Capacitor_SMD:C_0402_1005Metric" (id 2) (at 408.6352 204.47 0)
-      (effects (font (size 1.27 1.27)) hide)
-    )
+    (property "Footprint" "qsbc:C_0402_1005Metric" (id 2) (at 408.6352 204.47 0)
+      (effects (font (size 1.27 1.27)) hide)
+    )

Commit message: swap usb ctrl signals for layout
Parts:
- TP10, TP11, TP12, TP13, TP14, TP15, TP16, TP17, TP18, TP19, TP2, TP20, TP3, TP4, TP5, TP6, TP7, TP8, TP9: footprint TestPoint:TestPoint_Pad_D1.0mm -> qsbc:TestPoint_Pad_D0.4mm
Changed lines of the file:
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@@
       (effects (font (size 1.27 1.27)) (justify left))
     )
-    (property "Footprint" "TestPoint:TestPoint_Pad_D1.0mm" (id 2) (at 262.89 49.53 0)
+    (property "Footprint" "qsbc:TestPoint_Pad_D0.4mm" (id 2) (at 262.89 49.53 0)
       (effects (font (size 1.27 1.27)) hide)
     )
@@
       (effects (font (size 1.27 1.27)) (justify left))
     )
-    (property "Footprint" "TestPoint:TestPoint_Pad_D1.0mm" (id 2) (at 78.74 381 0)
+    (property "Footprint" "qsbc:TestPoint_Pad_D0.4mm" (id 2) (at 78.74 381 0)
       (effects (font (size 1.27 1.27)) hide)
     )
@@
       (effects (font (size 1.27 1.27)) (justify left))
     )
-    (property "Footprint" "TestPoint:TestPoint_Pad_D1.0mm" (id 2) (at 226.06 281.94 0)
+    (property "Footprint" "qsbc:TestPoint_Pad_D0.4mm" (id 2) (at 226.06 281.94 0)
       (effects (font (size 1.27 1.27)) hide)
     )
@@
       (effects (font (size 1.27 1.27)) (justify left))
     )
-    (property "Footprint" "TestPoint:TestPoint_Pad_D1.0mm" (id 2) (at 226.06 226.06 0)
+    (property "Footprint" "qsbc:TestPoint_Pad_D0.4mm" (id 2) (at 226.06 226.06 0)
       (effects (font (size 1.27 1.27)) hide)
     )
@@
       (effects (font (size 1.27 1.27)) (justify left))
     )
-    (property "Footprint" "TestPoint:TestPoint_Pad_D1.0mm" (id 2) (at 64.77 381 0)
+    (property "Footprint" "qsbc:TestPoint_Pad_D0.4mm" (id 2) (at 64.77 381 0)
       (effects (font (size 1.27 1.27)) hide)
     )
@@
       (effects (font (size 1.27 1.27)) (justify left))
     )
-    (property "Footprint" "TestPoint:TestPoint_Pad_D1.0mm" (id 2) (at 50.8 381 0)
+    (property "Footprint" "qsbc:TestPoint_Pad_D0.4mm" (id 2) (at 50.8 381 0)
       (effects (font (size 1.27 1.27)) hide)
     )
@@
       (effects (font (size 1.27 1.27)) (justify left))
     )
-    (property "Footprint" "TestPoint:TestPoint_Pad_D1.0mm" (id 2) (at 226.06 299.72 0)
+    (property "Footprint" "qsbc:TestPoint_Pad_D0.4mm" (id 2) (at 226.06 299.72 0)
       (effects (font (size 1.27 1.27)) hide)
     )
@@
       (effects (font (size 1.27 1.27)) (justify left))
     )
-    (property "Footprint" "TestPoint:TestPoint_Pad_D1.0mm" (id 2) (at 219.71 102.87 0)
+    (property "Footprint" "qsbc:TestPoint_Pad_D0.4mm" (id 2) (at 219.71 102.87 0)
       (effects (font (size 1.27 1.27)) hide)
     )
@@
       (effects (font (size 1.27 1.27)) (justify left))
     )
-    (property "Footprint" "TestPoint:TestPoint_Pad_D1.0mm" (id 2) (at 262.89 82.55 0)
+    (property "Footprint" "qsbc:TestPoint_Pad_D0.4mm" (id 2) (at 262.89 82.55 0)
       (effects (font (size 1.27 1.27)) hide)
     )
@@
       (effects (font (size 1.27 1.27)) (justify left))
     )
-    (property "Footprint" "TestPoint:TestPoint_Pad_D1.0mm" (id 2) (at 226.06 261.62 0)
+    (property "Footprint" "qsbc:TestPoint_Pad_D0.4mm" (id 2) (at 226.06 261.62 0)
       (effects (font (size 1.27 1.27)) hide)
     )
@@
       (effects (font (size 1.27 1.27)) (justify left))
     )
-    (property "Footprint" "TestPoint:TestPoint_Pad_D1.0mm" (id 2) (at 226.06 190.5 0)
+    (property "Footprint" "qsbc:TestPoint_Pad_D0.4mm" (id 2) (at 226.06 190.5 0)
       (effects (font (size 1.27 1.27)) hide)
     )
@@
       (effects (font (size 1.27 1.27)) (justify left))
     )
-    (property "Footprint" "TestPoint:TestPoint_Pad_D1.0mm" (id 2) (at 219.71 120.65 0)
+    (property "Footprint" "qsbc:TestPoint_Pad_D0.4mm" (id 2) (at 219.71 120.65 0)
       (effects (font (size 1.27 1.27)) hide)
     )
@@
       (effects (font (size 1.27 1.27)) (justify left))
     )
-    (property "Footprint" "TestPoint:TestPoint_Pad_D1.0mm" (id 2) (at 262.89 64.77 0)
+    (property "Footprint" "qsbc:TestPoint_Pad_D0.4mm" (id 2) (at 262.89 64.77 0)
       (effects (font (size 1.27 1.27)) hide)
     )
@@
       (effects (font (size 1.27 1.27)) (justify left))
     )
-    (property "Footprint" "TestPoint:TestPoint_Pad_D1.0mm" (id 2) (at 226.06 208.28 0)
+    (property "Footprint" "qsbc:TestPoint_Pad_D0.4mm" (id 2) (at 226.06 208.28 0)
       (effects (font (size 1.27 1.27)) hide)
     )
@@
       (effects (font (size 1.27 1.27)) (justify left))
     )
-    (property "Footprint" "TestPoint:TestPoint_Pad_D1.0mm" (id 2) (at 92.71 381 0)
+    (property "Footprint" "qsbc:TestPoint_Pad_D0.4mm" (id 2) (at 92.71 381 0)
       (effects (font (size 1.27 1.27)) hide)
     )
@@
       (effects (font (size 1.27 1.27)) (justify left))
     )
-    (property "Footprint" "TestPoint:TestPoint_Pad_D1.0mm" (id 2) (at 226.06 243.84 0)
+    (property "Footprint" "qsbc:TestPoint_Pad_D0.4mm" (id 2) (at 226.06 243.84 0)
       (effects (font (size 1.27 1.27)) hide)
     )
@@
       (effects (font (size 1.27 1.27)) (justify left))
     )
-    (property "Footprint" "TestPoint:TestPoint_Pad_D1.0mm" (id 2) (at 312.42 212.09 0)
+    (property "Footprint" "qsbc:TestPoint_Pad_D0.4mm" (id 2) (at 312.42 212.09 0)
       (effects (font (size 1.27 1.27)) hide)
     )
@@
       (effects (font (size 1.27 1.27)) (justify left))
     )
-    (property "Footprint" "TestPoint:TestPoint_Pad_D1.0mm" (id 2) (at 326.39 213.36 0)
+    (property "Footprint" "qsbc:TestPoint_Pad_D0.4mm" (id 2) (at 326.39 213.36 0)
       (effects (font (size 1.27 1.27)) hide)
     )
@@
       (effects (font (size 1.27 1.27)) (justify left))
     )
-    (property "Footprint" "TestPoint:TestPoint_Pad_D1.0mm" (id 2) (at 219.71 138.43 0)
-      (effects (font (size 1.27 1.27)) hide)
-    )
+    (property "Footprint" "qsbc:TestPoint_Pad_D0.4mm" (id 2) (at 219.71 138.43 0)
+      (effects (font (size 1.27 1.27)) hide)
+    )

Commit message: pmic routing almost done
Parts:
- C64, C65, C66, C67, C68, C69, C70, C71, C78, C79, C80, C81, C82, C83, C84, C85, C86, C87, C88, C89, C91: footprint Capacitor_SMD:C_0603_1608Metric -> qsbc:C_0603_1608Metric
Connections:
- net NVCC_DRAM_1.1V is gone; now on net VDD_DRAM_1.1V: U3.38 (BUCK8_FB)
Changed lines of the file:
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@@
     (effects (font (size 1.27 1.27)) (justify left bottom))
   )
-  (label "NVCC_DRAM_1.1V" (at 173.99 146.05 0)
+  (label "VDD_DRAM_1.1V" (at 173.99 146.05 0)
     (effects (font (size 1.27 1.27)) (justify left bottom))
   )
@@
       (effects (font (size 1.27 1.27)) (justify left))
     )
-    (property "Footprint" "Capacitor_SMD:C_0603_1608Metric" (id 2) (at 252.4252 133.35 0)
+    (property "Footprint" "qsbc:C_0603_1608Metric" (id 2) (at 252.4252 133.35 0)
       (effects (font (size 1.27 1.27)) hide)
     )
@@
       (effects (font (size 1.27 1.27)) (justify left))
     )
-    (property "Footprint" "Capacitor_SMD:C_0603_1608Metric" (id 2) (at 300.6852 95.25 0)
+    (property "Footprint" "qsbc:C_0603_1608Metric" (id 2) (at 300.6852 95.25 0)
       (effects (font (size 1.27 1.27)) hide)
     )
@@
       (effects (font (size 1.27 1.27)) (justify left))
     )
-    (property "Footprint" "Capacitor_SMD:C_0603_1608Metric" (id 2) (at 116.5352 130.81 0)
+    (property "Footprint" "qsbc:C_0603_1608Metric" (id 2) (at 116.5352 130.81 0)
       (effects (font (size 1.27 1.27)) hide)
     )
@@
       (effects (font (size 1.27 1.27)) (justify left))
     )
-    (property "Footprint" "Capacitor_SMD:C_0603_1608Metric" (id 2) (at 270.2052 115.57 0)
+    (property "Footprint" "qsbc:C_0603_1608Metric" (id 2) (at 270.2052 115.57 0)
       (effects (font (size 1.27 1.27)) hide)
     )
@@
       (effects (font (size 1.27 1.27)) (justify left))
     )
-    (property "Footprint" "Capacitor_SMD:C_0603_1608Metric" (id 2) (at 318.4652 77.47 0)
+    (property "Footprint" "qsbc:C_0603_1608Metric" (id 2) (at 318.4652 77.47 0)
       (effects (font (size 1.27 1.27)) hide)
     )
@@
       (effects (font (size 1.27 1.27)) (justify left))
     )
-    (property "Footprint" "Capacitor_SMD:C_0603_1608Metric" (id 2) (at 116.5352 148.59 0)
+    (property "Footprint" "qsbc:C_0603_1608Metric" (id 2) (at 116.5352 148.59 0)
       (effects (font (size 1.27 1.27)) hide)
     )
@@
       (effects (font (size 1.27 1.27)) (justify left))
     )
-    (property "Footprint" "Capacitor_SMD:C_0603_1608Metric" (id 2) (at 116.5352 110.49 0)
+    (property "Footprint" "qsbc:C_0603_1608Metric" (id 2) (at 116.5352 110.49 0)
       (effects (font (size 1.27 1.27)) hide)
     )
@@
       (effects (font (size 1.27 1.27)) (justify left))
     )
-    (property "Footprint" "Capacitor_SMD:C_0603_1608Metric" (id 2) (at 336.2452 62.23 0)
+    (property "Footprint" "qsbc:C_0603_1608Metric" (id 2) (at 336.2452 62.23 0)
       (effects (font (size 1.27 1.27)) hide)
     )
@@
       (effects (font (size 1.27 1.27)) (justify left))
     )
-    (property "Footprint" "Capacitor_SMD:C_0603_1608Metric" (id 2) (at 103.8352 59.69 0)
+    (property "Footprint" "qsbc:C_0603_1608Metric" (id 2) (at 103.8352 59.69 0)
       (effects (font (size 1.27 1.27)) hide)
     )
@@
       (effects (font (size 1.27 1.27)) (justify left))
     )
-    (property "Footprint" "Capacitor_SMD:C_0603_1608Metric" (id 2) (at 282.9052 115.57 0)
+    (property "Footprint" "qsbc:C_0603_1608Metric" (id 2) (at 282.9052 115.57 0)
       (effects (font (size 1.27 1.27)) hide)
     )
@@
       (effects (font (size 1.27 1.27)) (justify left))
     )
-    (property "Footprint" "Capacitor_SMD:C_0603_1608Metric" (id 2) (at 116.5352 59.69 0)
+    (property "Footprint" "qsbc:C_0603_1608Metric" (id 2) (at 116.5352 59.69 0)
       (effects (font (size 1.27 1.27)) hide)
     )
@@
       (effects (font (size 1.27 1.27)) (justify left))
     )
-    (property "Footprint" "Capacitor_SMD:C_0603_1608Metric" (id 2) (at 103.8352 110.49 0)
+    (property "Footprint" "qsbc:C_0603_1608Metric" (id 2) (at 103.8352 110.49 0)
       (effects (font (size 1.27 1.27)) hide)
     )
@@
       (effects (font (size 1.27 1.27)) (justify left))
     )
-    (property "Footprint" "Capacitor_SMD:C_0603_1608Metric" (id 2) (at 287.9852 95.25 0)
+    (property "Footprint" "qsbc:C_0603_1608Metric" (id 2) (at 287.9852 95.25 0)
       (effects (font (size 1.27 1.27)) hide)
     )
@@
       (effects (font (size 1.27 1.27)) (justify left))
     )
-    (property "Footprint" "Capacitor_SMD:C_0603_1608Metric" (id 2) (at 305.7652 77.47 0)
+    (property "Footprint" "qsbc:C_0603_1608Metric" (id 2) (at 305.7652 77.47 0)
       (effects (font (size 1.27 1.27)) hide)
     )
@@
       (effects (font (size 1.27 1.27)) (justify left))
     )
-    (property "Footprint" "Capacitor_SMD:C_0603_1608Metric" (id 2) (at 228.2952 151.13 0)
+    (property "Footprint" "qsbc:C_0603_1608Metric" (id 2) (at 228.2952 151.13 0)
       (effects (font (size 1.27 1.27)) hide)
     )
@@
       (effects (font (size 1.27 1.27)) (justify left))
     )
-    (property "Footprint" "Capacitor_SMD:C_0603_1608Metric" (id 2) (at 215.5952 151.13 0)
+    (property "Footprint" "qsbc:C_0603_1608Metric" (id 2) (at 215.5952 151.13 0)
       (effects (font (size 1.27 1.27)) hide)
     )
@@
       (effects (font (size 1.27 1.27)) (justify left))
     )
-    (property "Footprint" "Capacitor_SMD:C_0603_1608Metric" (id 2) (at 265.1252 133.35 0)
+    (property "Footprint" "qsbc:C_0603_1608Metric" (id 2) (at 265.1252 133.35 0)
       (effects (font (size 1.27 1.27)) hide)
     )
@@
       (effects (font (size 1.27 1.27)) (justify left))
     )
-    (property "Footprint" "Capacitor_SMD:C_0603_1608Metric" (id 2) (at 323.5452 62.23 0)
+    (property "Footprint" "qsbc:C_0603_1608Metric" (id 2) (at 323.5452 62.23 0)
       (effects (font (size 1.27 1.27)) hide)
     )
@@
       (effects (font (size 1.27 1.27)) (justify left))
     )
-    (property "Footprint" "Capacitor_SMD:C_0603_1608Metric" (id 2) (at 116.5352 90.17 0)
+    (property "Footprint" "qsbc:C_0603_1608Metric" (id 2) (at 116.5352 90.17 0)
       (effects (font (size 1.27 1.27)) hide)
     )
@@
       (effects (font (size 1.27 1.27)) (justify left))
     )
-    (property "Footprint" "Capacitor_SMD:C_0603_1608Metric" (id 2) (at 195.2752 311.15 0)
+    (property "Footprint" "qsbc:C_0603_1608Metric" (id 2) (at 195.2752 311.15 0)
       (effects (font (size 1.27 1.27)) hide)
     )
@@
       (effects (font (size 1.27 1.27)) (justify left))
     )
-    (property "Footprint" "Capacitor_SMD:C_0603_1608Metric" (id 2) (at 116.5352 74.93 0)
-      (effects (font (size 1.27 1.27)) hide)
-    )
+    (property "Footprint" "qsbc:C_0603_1608Metric" (id 2) (at 116.5352 74.93 0)
+      (effects (font (size 1.27 1.27)) hide)
+    )
