File: power.kicad_sch (KiCad schematic)
At the start: 71 parts, among them SW1 SW_Push, U3 BD71847MWV, Y1 32.768Khz

Commit message: misc bom cleanup
Parts:
- R13: DNP (none) -> DNP
Changed lines of the file:
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@@
       (effects (font (size 1.27 1.27)) hide)
+    )
+    (property "DNP" "DNP" (at 341.63 157.48 90)
+      (effects (font (size 1.27 1.27)))
     )
     (pin "1")
