File: misc.kicad_sch (KiCad schematic)
At the start: 25 parts, among them J7 Conn_ARM_JTAG_SWD_10, SW2 SW_DIP_x02, U1 MIMX8MM6DVTLZAA, Y3 24Mhz

Commit message: Rev 1
Parts:
- renumbered R101 to R100, R102 to R101, R103 to R102, R104 to R103, R105 to R104, R106 to R105, R107 to R106, R108 to R107, R96 to R95, R97 to R96, R98 to R97, R99 to R98, R100 to R99, TP22 to TP23, TP23 to TP24, TP24 to TP25, TP25 to TP26, TP26 to TP27
Changed lines of the file:
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@@
   (title_block
     (title "QSBC")
-    (rev "1")
+    (date "2022-12-01")
+    (rev "1.0")
     (company "Q-LAB")
   )
@@
   (symbol (lib_id "Device:R") (at 224.79 104.14 0) (unit 1)
     (in_bom yes) (on_board yes)
-    (property "Reference" "R105" (id 0) (at 227.33 102.8699 0)
+    (property "Reference" "R104" (id 0) (at 227.33 102.8699 0)
       (effects (font (size 1.27 1.27)) (justify left))
     )
@@
   (symbol (lib_id "power:GND") (at 129.54 185.42 0) (unit 1)
     (in_bom yes) (on_board yes) (fields_autoplaced)
-    (property "Reference" "#PWR0139" (id 0) (at 129.54 191.77 0)
+    (property "Reference" "#PWR0138" (id 0) (at 129.54 191.77 0)
       (effects (font (size 1.27 1.27)) hide)
     )
@@
   (symbol (lib_id "Connector:TestPoint") (at 256.54 87.63 270) (unit 1)
     (in_bom no) (on_board yes) (fields_autoplaced)
-    (property "Reference" "TP26" (id 0) (at 261.62 86.3599 90)
+    (property "Reference" "TP27" (id 0) (at 261.62 86.3599 90)
       (effects (font (size 1.27 1.27)) (justify left))
     )
@@
   (symbol (lib_id "Device:R") (at 214.63 35.56 0) (unit 1)
     (in_bom yes) (on_board yes)
-    (property "Reference" "R103" (id 0) (at 217.17 34.2899 0)
+    (property "Reference" "R102" (id 0) (at 217.17 34.2899 0)
       (effects (font (size 1.27 1.27)) (justify left))
     )
@@
   (symbol (lib_id "Device:R") (at 234.95 35.56 0) (unit 1)
     (in_bom yes) (on_board yes)
-    (property "Reference" "R106" (id 0) (at 237.49 34.2899 0)
+    (property "Reference" "R105" (id 0) (at 237.49 34.2899 0)
       (effects (font (size 1.27 1.27)) (justify left))
     )
@@
   (symbol (lib_id "Connector:TestPoint") (at 81.28 64.77 0) (unit 1)
     (in_bom no) (on_board yes) (fields_autoplaced)
-    (property "Reference" "TP25" (id 0) (at 83.82 60.1979 0)
+    (property "Reference" "TP26" (id 0) (at 83.82 60.1979 0)
       (effects (font (size 1.27 1.27)) (justify left))
     )
@@
   (symbol (lib_id "Device:R") (at 204.47 35.56 0) (unit 1)
     (in_bom yes) (on_board yes)
-    (property "Reference" "R101" (id 0) (at 207.01 34.2899 0)
+    (property "Reference" "R100" (id 0) (at 207.01 34.2899 0)
       (effects (font (size 1.27 1.27)) (justify left))
     )
@@
   (symbol (lib_id "Device:R") (at 96.52 58.42 0) (unit 1)
     (in_bom yes) (on_board yes)
-    (property "Reference" "R96" (id 0) (at 99.06 57.1499 0)
+    (property "Reference" "R95" (id 0) (at 99.06 57.1499 0)
       (effects (font (size 1.27 1.27)) (justify left))
     )
@@
   (symbol (lib_id "Device:R") (at 109.22 111.76 90) (unit 1)
     (in_bom yes) (on_board yes)
-    (property "Reference" "R99" (id 0) (at 109.22 105.41 90))
+    (property "Reference" "R98" (id 0) (at 109.22 105.41 90))
     (property "Value" "510K" (id 1) (at 109.22 107.95 90))
     (property "Footprint" "qsbc:R_0402_1005Metric" (id 2) (at 109.22 113.538 90)
@@
   (symbol (lib_id "power:GND") (at 109.22 140.97 0) (unit 1)
     (in_bom yes) (on_board yes) (fields_autoplaced)
-    (property "Reference" "#PWR0138" (id 0) (at 109.22 147.32 0)
+    (property "Reference" "#PWR0137" (id 0) (at 109.22 147.32 0)
       (effects (font (size 1.27 1.27)) hide)
     )
@@
   (symbol (lib_id "Connector:TestPoint") (at 68.58 64.77 0) (unit 1)
     (in_bom no) (on_board yes) (fields_autoplaced)
-    (property "Reference" "TP24" (id 0) (at 71.12 60.1979 0)
+    (property "Reference" "TP25" (id 0) (at 71.12 60.1979 0)
       (effects (font (size 1.27 1.27)) (justify left))
     )
@@
   (symbol (lib_id "Device:R") (at 234.95 104.14 0) (unit 1)
     (in_bom yes) (on_board yes)
-    (property "Reference" "R107" (id 0) (at 237.49 102.8699 0)
+    (property "Reference" "R106" (id 0) (at 237.49 102.8699 0)
       (effects (font (size 1.27 1.27)) (justify left))
     )
@@
   (symbol (lib_id "Device:R") (at 214.63 104.14 0) (unit 1)
     (in_bom yes) (on_board yes)
-    (property "Reference" "R104" (id 0) (at 217.17 102.8699 0)
+    (property "Reference" "R103" (id 0) (at 217.17 102.8699 0)
       (effects (font (size 1.27 1.27)) (justify left))
     )
@@
   (symbol (lib_id "Device:R") (at 116.84 58.42 0) (unit 1)
     (in_bom yes) (on_board yes)
-    (property "Reference" "R100" (id 0) (at 119.38 57.1499 0)
+    (property "Reference" "R99" (id 0) (at 119.38 57.1499 0)
       (effects (font (size 1.27 1.27)) (justify left))
     )
@@
   (symbol (lib_id "power:GND") (at 234.95 113.03 0) (unit 1)
     (in_bom yes) (on_board yes) (fields_autoplaced)
-    (property "Reference" "#PWR0140" (id 0) (at 234.95 119.38 0)
+    (property "Reference" "#PWR0139" (id 0) (at 234.95 119.38 0)
       (effects (font (size 1.27 1.27)) hide)
     )
@@
   (symbol (lib_id "Device:R") (at 204.47 104.14 0) (unit 1)
     (in_bom yes) (on_board yes)
-    (property "Reference" "R102" (id 0) (at 207.01 102.8699 0)
+    (property "Reference" "R101" (id 0) (at 207.01 102.8699 0)
       (effects (font (size 1.27 1.27)) (justify left))
     )
@@
   (symbol (lib_id "Device:R") (at 245.11 81.28 0) (unit 1)
     (in_bom yes) (on_board yes)
-    (property "Reference" "R108" (id 0) (at 247.65 80.0099 0)
+    (property "Reference" "R107" (id 0) (at 247.65 80.0099 0)
       (effects (font (size 1.27 1.27)) (justify left))
     )
@@
   (symbol (lib_id "Connector:TestPoint") (at 43.18 64.77 0) (unit 1)
     (in_bom no) (on_board yes) (fields_autoplaced)
-    (property "Reference" "TP22" (id 0) (at 45.72 60.1979 0)
+    (property "Reference" "TP23" (id 0) (at 45.72 60.1979 0)
       (effects (font (size 1.27 1.27)) (justify left))
     )
@@
   (symbol (lib_id "Device:R") (at 106.68 58.42 0) (unit 1)
     (in_bom yes) (on_board yes)
-    (property "Reference" "R97" (id 0) (at 109.22 57.1499 0)
+    (property "Reference" "R96" (id 0) (at 109.22 57.1499 0)
       (effects (font (size 1.27 1.27)) (justify left))
     )
@@
   (symbol (lib_id "Device:R") (at 107.95 91.44 90) (unit 1)
     (in_bom yes) (on_board yes) (fields_autoplaced)
-    (property "Reference" "R98" (id 0) (at 107.95 85.09 90))
+    (property "Reference" "R97" (id 0) (at 107.95 85.09 90))
     (property "Value" "0R" (id 1) (at 107.95 87.63 90))
     (property "Footprint" "qsbc:R_0402_1005Metric" (id 2) (at 107.95 93.218 90)
@@
   (symbol (lib_id "Connector:TestPoint") (at 55.88 64.77 0) (unit 1)
     (in_bom no) (on_board yes) (fields_autoplaced)
-    (property "Reference" "TP23" (id 0) (at 58.42 60.1979 0)
-      (effects (font (size 1.27 1.27)) (justify left))
-    )
+    (property "Reference" "TP24" (id 0) (at 58.42 60.1979 0)
+      (effects (font (size 1.27 1.27)) (justify left))
+    )

Commit message: misc changes for rev1
Parts:
- J7, R105: now left out of the parts list
Changed lines of the file:
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@@
   )
   (symbol (lib_id "Device:R") (at 234.95 35.56 0) (unit 1)
-    (in_bom yes) (on_board yes)
+    (in_bom no) (on_board yes)
     (property "Reference" "R105" (id 0) (at 237.49 34.2899 0)
       (effects (font (size 1.27 1.27)) (justify left))
@@
   )
   (symbol (lib_id "Connector:Conn_ARM_JTAG_SWD_10") (at 129.54 165.1 0) (unit 1)
-    (in_bom yes) (on_board yes)
+    (in_bom no) (on_board yes)
     (property "Reference" "J7" (id 0) (at 121.92 151.13 0)
       (effects (font (size 1.27 1.27)) (justify right))
