File: imx8mm_power.kicad_sch (KiCad schematic)
At the start: 57 parts, among them U1 MIMX8MM6DVTLZAA

Commit message: misc bom cleanup
Changed lines of the file:
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@@
     (stroke (width 0) (type default))
   )
-  (wire (pts (xy 54.61 162.56) (xy 77.47 162.56))
+  (wire (pts (xy 40.64 162.56) (xy 77.47 162.56))
     (stroke (width 0) (type default))
   )
@@
     (effects (font (size 1.27 1.27)) (justify left bottom))
   )
-  (label "VDD_DRAM_xPU_0.9V" (at 54.61 162.56 0) (fields_autoplaced)
+  (label "VDD_DRAM_xPU_0.9V" (at 40.64 162.56 0) (fields_autoplaced)
     (effects (font (size 1.27 1.27)) (justify left bottom))
   )
